File: EPSv1.kicad_pcb (KiCad board)
At the start: 2 copper layers, 50 x 100 mm, 34 parts, among them J1 Conn_01x04, Q1 AO3400A, Q2 AO3400A, Q3 AO3400A, Q4 AO3400A, U1 BQ29700DSER, U2 BQ29700DSER, U3 MCP73831T-2ACI/OT, U4 MCP73831T-2ACI/OT

Commit message: Laid out all the blocks and imported the board outline
Parts:
- removed the J1 at (159.5, 65.2)
- added H1: MountingHole_Pad, MountingHole:MountingHole_2.7mm_M2.5_Pad_Via, F.Cu at (30.7, 0.00)
- added H10: MountingHole_Pad, MountingHole:MountingHole_2.7mm_M2.5_Pad_Via, F.Cu at (-25.2, -20.3)
- added H11: MountingHole_Pad, MountingHole:MountingHole_2.7mm_M2.5_Pad_Via, F.Cu at (-16.8, -27.4)
- added H12: MountingHole_Pad, MountingHole:MountingHole_2.7mm_M2.5_Pad_Via, F.Cu at (-6.49, -31.2)
- added H13: MountingHole_Pad, MountingHole:MountingHole_2.7mm_M2.5_Pad_Via, F.Cu at (4.50, -31.2)
- added H14: MountingHole_Pad, MountingHole:MountingHole_2.7mm_M2.5_Pad_Via, F.Cu at (23.3, -20.3)
- added H15: MountingHole_Pad, MountingHole:MountingHole_2.7mm_M2.5_Pad_Via, F.Cu at (28.7, -10.8)
- added H2: MountingHole_Pad, MountingHole:MountingHole_2.7mm_M2.5_Pad_Via, F.Cu at (28.7, 10.8)
- added H3: MountingHole_Pad, MountingHole:MountingHole_2.7mm_M2.5_Pad_Via, F.Cu at (23.3, 20.3)
- added H4: MountingHole_Pad, MountingHole:MountingHole_2.7mm_M2.5_Pad_Via, F.Cu at (4.50, 31.2)
- added H5: MountingHole_Pad, MountingHole:MountingHole_2.7mm_M2.5_Pad_Via, F.Cu at (-6.49, 31.2)
- added H6: MountingHole_Pad, MountingHole:MountingHole_2.7mm_M2.5_Pad_Via, F.Cu at (-16.8, 27.4)
- added H7: MountingHole_Pad, MountingHole:MountingHole_2.7mm_M2.5_Pad_Via, F.Cu at (-25.2, 20.3)
- added H8: MountingHole_Pad, MountingHole:MountingHole_2.7mm_M2.5_Pad_Via, F.Cu at (-30.7, 10.8)
- added H9: MountingHole_Pad, MountingHole:MountingHole_2.7mm_M2.5_Pad_Via, F.Cu at (-30.7, -10.8)
- added J1: Conn_01x04, Rocketry_Manual:1054301102, F.Cu at (-21.1, 0.00)
- added J1: Conn_01x04, Rocketry_Manual:1054301102, F.Cu at (8.64, 17.3)
- added J1: Conn_01x04, Rocketry_Manual:1054301102, F.Cu at (-74.9, 19.8)
- added R13: 100k 0603, Rocketry_Easyeda:R0603, F.Cu at (-9.73, -3.97)
- added R14: 100k 0603, Rocketry_Easyeda:R0603, F.Cu at (-10.6, -18.1)
- added R15: 100k 0603, Rocketry_Easyeda:R0603, F.Cu at (-16.5, -18.1)
- added U5: C3235556 (M66200DRLR), Rocketry_Easyeda:SOT-583-8_L2.1-W1.2-P0.50-LS1.6-BL, F.Cu at (-9.99, -1.43)
- added U6: C3235556 (M66200DRLR), Rocketry_Easyeda:SOT-583-8_L2.1-W1.2-P0.50-LS1.6-BL, F.Cu at (-10.7, -15.4)
- added U7: C3235556 (M66200DRLR), Rocketry_Easyeda:SOT-583-8_L2.1-W1.2-P0.50-LS1.6-BL, F.Cu at (-16.6, -15.4)
- moved BT2 235.4 mm to (-101.4, 71.4)
- moved BT1 235.4 mm to (-76.8, 71.4)
- moved USB1 230.6 mm to (-103.7, 21.1)
- moved LED1 38.3 mm to (-2.03, -9.98), turned to -90 degrees
- moved LED2 35.7 mm to (0.00, -10.7), turned to -90 degrees
- moved R10 31.6 mm to (-3.05, -4.10)
- moved C3 30.7 mm to (-3.81, -9.94), turned to -90 degrees
- moved U3 29.9 mm to (-0.98, -6.64), turned to 90 degrees
- moved R9 27.5 mm to (0.25, -3.84)
- moved R8 27.2 mm to (22.1, 3.56), turned to 180 degrees
- moved C4 27.1 mm to (2.03, -6.89), turned to 90 degrees
- moved R4 25.5 mm to (22.1, -6.86), turned to 180 degrees
- moved C2 24.2 mm to (23.3, 6.10), turned to 90 degrees
- moved LED3 22.5 mm to (-2.03, 1.96), turned to -90 degrees
- moved R7 22.5 mm to (21.6, 8.64), turned to -90 degrees
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- renumbered USB2 to USB1
Connections:
- net /MCP73831_1/+5V_VIN renamed /LM66200_1/VOUT
Routing:
- net GND: track 0.00 -> 3.72 mm, vias 0 -> 2
- net Net-(U5-ST): track 0.00 -> 3.43 mm
- net /LM66200_1/VIN1: track 0.00 -> 2.00 mm
- net /LM66200_1/VOUT: track 0.00 -> 1.28 mm
- added copper zone on B.Cu, net GND
- added copper zone on F.Cu, net GND
Other:
- board size 50 x 100 mm -> 148.1 x 148.8 mm

Commit message: 100x100 board size
Parts:
- removed H10, H11, H12, H13, H14, H15, H5, H6, H7, H8, H9: MountingHole_Pad, MountingHole:MountingHole_2.7mm_M2.5_Pad_Via
- removed the J1 at (-21.1, 0.00)
- removed the J1 at (8.64, 17.3)
- removed the J1 at (-74.9, 19.8)
- added C10: 10n, Capacitor_SMD:C_0402_1005Metric, F.Cu at (154.1, 14.5)
- added C11: 100n, Capacitor_SMD:C_0402_1005Metric, F.Cu at (154.1, 16.5)
- added C12: 4.7u, Capacitor_SMD:C_0402_1005Metric, F.Cu at (154.1, 18.5)
- added C7: 4.7u, Capacitor_SMD:C_0402_1005Metric, F.Cu at (154.1, 8.62)
- added C8: 100n, Capacitor_SMD:C_0402_1005Metric, F.Cu at (154.1, 10.6)
- added C9: 100n, Capacitor_SMD:C_0402_1005Metric, F.Cu at (154.1, 12.6)
- added J1: Molex_Microfit, Rocketry_Manual:1054301102, F.Cu at (93.7, 38.6)
- added J2: Conn_01x05_Pin, Connector_PinHeader_1.27mm:PinHeader_1x05_P1.27mm_Vertical, F.Cu at (204.1, 6.39)
- added J3: Molex_Microfit, Rocketry_Manual:1054301102, F.Cu at (93.7, 28.7)
- added J4: Molex_Microfit, Rocketry_Manual:1054301102, F.Cu at (93.7, 18.8)
- added R16: 100k 0603, Rocketry_Easyeda:R0603, F.Cu at (81.7, 16.7)
- added R17: 5.1K, Resistor_SMD:R_0402_1005Metric, F.Cu at (167.8, 8.63)
- added R18: 5.1K, Resistor_SMD:R_0402_1005Metric, F.Cu at (167.8, 10.6)
- added R19: 5.1K, Resistor_SMD:R_0402_1005Metric, F.Cu at (167.8, 12.6)
- added R20: 100k 0603, Rocketry_Easyeda:R0603, F.Cu at (81.7, 28.2)
- added R21: 100k 0603, Rocketry_Easyeda:R0603, F.Cu at (81.7, 38.6)
- added U10: MCP9700AT-E/TT, Rocketry_Easyeda:SOT-23-3_L2.9-W1.3-P1.90-LS2.4-BR, F.Cu at (51.1, 74.4)
- added U11: C3235556 (M66200DRLR), Rocketry_Easyeda:SOT-583-8_L2.1-W1.2-P0.50-LS1.6-BL, F.Cu at (81.5, 30.9)
- added U12: C3235556 (M66200DRLR), Rocketry_Easyeda:SOT-583-8_L2.1-W1.2-P0.50-LS1.6-BL, F.Cu at (81.5, 41.3)
- added U8: C3235556 (M66200DRLR), Rocketry_Easyeda:SOT-583-8_L2.1-W1.2-P0.50-LS1.6-BL, F.Cu at (81.6, 19.4)
- added U9: STM32L432KCUx, Package_DFN_QFN:QFN-32-1EP_5x5mm_P0.5mm_EP3.45x3.45mm, F.Cu at (58.0, 29.2)
- added USB2: TYPE-C 16PIN 2MD(073), Rocketry_Easyeda:USB-C-SMD_TYPE-C-6PIN-2MD-073, F.Cu at (6.08, 13.2)
- moved BT2 153.2 mm to (51.1, 86.6), turned to 0 degrees
- moved R14 149.3 mm to (136.2, -45.6)
- moved R15 149.3 mm to (130.2, -45.6)
- moved U6 149.3 mm to (136.0, -42.9)
- moved U7 149.3 mm to (130.1, -42.9)
- moved R13 129.4 mm to (119.5, 2.27)
- moved U5 129.4 mm to (119.3, 4.81)
- moved BT1 128.2 mm to (51.1, 62.0), turned to 0 degrees
- moved H4 113.2 mm to (96.8, 96.8)
- moved H3 79.0 mm to (3.30, 96.8)
- moved H2 68.4 mm to (96.8, 3.30)
- moved C4 39.1 mm to (12.7, 30.7)
- moved C5 39.1 mm to (6.86, 39.6)
- moved LED4 39.1 mm to (10.7, 38.9)
- moved R12 39.1 mm to (7.62, 45.5)
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Connections:
- R14 pad 2: /LM66200_2/VIN1 -> /BQ29700_1/CELL+
- U6 pad 3: /LM66200_2/VIN1 -> /BQ29700_1/CELL+
- U6 pad 6: /LM66200_2/VIN2 -> /BQ29700_2/CELL+
Routing:
- net /BQ29700_1/CELL+: track 0.00 -> 2.74 mm
- net /LM66200_1/VIN1: track 2.00 -> 4.59 mm
- net /LM66200_1/VIN2: track 0.00 -> 2.42 mm
- net /LM66200_1/VOUT: track 1.28 -> 3.58 mm
- net GND: track 3.72 -> 3.05 mm
- added copper zone on F.Cu, net /LM66200_1/VIN1
- added copper zone on F.Cu, net Net-(U5-ST)
Other:
- board size 148.1 x 148.8 mm -> 199.4 x 114.2 mm
- copper layers 2 -> 4

Commit message: adde new blocks
Parts:
- added C13: 10uF 0603, Rocketry_Easyeda:C0603, F.Cu at (24.1, -12.7)
- added C14: 10uF 0603, Rocketry_Easyeda:C0603, F.Cu at (25.9, -12.7)
- added C15: 10uF 0603, Rocketry_Easyeda:C0603, F.Cu at (27.7, -12.7)
- added C16: 100nF 0603, Rocketry_Easyeda:C0603, F.Cu at (33.3, -10.1)
- added C17: 22uF 0805, Rocketry_Easyeda:C0805, F.Cu at (36.3, -14.7)
- added C18: 22uF 0805, Rocketry_Easyeda:C0805, F.Cu at (38.4, -14.7)
- added C19: 22uF 0805, Rocketry_Easyeda:C0805, F.Cu at (40.4, -14.7)
- added D1: BZT52C11-7-F, Rocketry_Easyeda:SOD-123_L2.8-W1.8-LS3.7-RD, F.Cu at (154.2, 81.8)
- added LED6: 0805G (Green), Rocketry_Easyeda:LED0805-R-RD, F.Cu at (36.1, -6.81)
- added LED7: KT-0603R (RED), Rocketry_Easyeda:LED0603-RD, F.Cu at (159.8, 72.4)
- added Q5: AP25P06K, Rocketry_Easyeda:TO-252-2_L6.6-W6.1-P4.57-LS10.1-BL, F.Cu at (154.9, 77.0)
- added R1: 470k 0603, Rocketry_Easyeda:R0603, F.Cu at (-7.37, 71.2)
- added R2: 470k 0603, Rocketry_Easyeda:R0603, F.Cu at (-7.37, 73.7)
- added R26: 0603WAF1001T5E (1k 0603), Rocketry_Easyeda:R0603, F.Cu at (156.7, 72.4)
- added R27: 0603WAF1003T5E (100k 0603), Rocketry_Easyeda:R0603, F.Cu at (158.2, 81.8)
- added R28: 10k 0603, Rocketry_Easyeda:R0603, F.Cu at (29.5, -12.7)
- added R29: 470k 0603, Rocketry_Easyeda:R0603, F.Cu at (35.8, -11.2)
- added R3: 470k 0603, Rocketry_Easyeda:R0603, F.Cu at (-7.37, 76.1)
- added R30: 150k 0603, Rocketry_Easyeda:R0603, F.Cu at (38.1, -10.4)
- added R31: 330R 0603, Rocketry_Easyeda:R0603, F.Cu at (38.1, -7.57)
- added R4: 470k 0603, Rocketry_Easyeda:R0603, F.Cu at (-7.37, 78.6)
- added U1: MCP9700AT-E/TT, Rocketry_Easyeda:SOT-23-3_L2.9-W1.3-P1.90-LS2.4-BR, F.Cu at (130.6, 44.3)
- added U14: 1.5uF 2.9A, Rocketry_Easyeda:IND-SMD_L2.5-W2.0_MEKK2520TR47M, F.Cu at (32.5, -16.2)
- added U15: TPS63070RNMR, Rocketry_Easyeda:VQFN-HR-15_L3.0-W2.5-P0.50-BL_TPS63070RNMR, F.Cu at (32.5, -12.7)
- moved J4 148.5 mm to (55.6, 3.30), turned to 90 degrees
- moved USB1 85.1 mm to (15.4, 4.06)
- renumbered J4 to J1, J3 to J2, J1 to J3, J2 to J4, R6 to R10, R7 to R11, R8 to R12, R9 to R13, R10 to R14, R11 to R15, R12 to R16, R13 to R17, R14 to R18, R15 to R19, R16 to R20, R17 to R21, R18 to R22, R19 to R23, R20 to R24, R21 to R25, R1 to R5, R2 to R6, R3 to R7, R4 to R8, R5 to R9, U8 to U10, U9 to U11, U11 to U12, U12 to U13, U10 to U2, U1 to U3, U2 to U4, U3 to U5, U4 to U6, U5 to U7, U6 to U8, U7 to U9
Connections:
- net /BQ29700_1/CELL+ renamed CELL_1+
- net /BQ29700_2/CELL+ renamed CELL_2+
- net /STM32L432KCUx/+3V3 renamed +3.3V
- U11 pad 11: /STM32L432KCUx/PA5 -> ~{MCU_LS_1}
- U11 pad 12: /STM32L432KCUx/PA6 -> ~{MCU_LS_2}
- U11 pad 13: /STM32L432KCUx/PA7 -> ~{MCU_LS_3}
- U11 pad 14: /STM32L432KCUx/PB0 -> PB0
- U11 pad 15: /STM32L432KCUx/PB1 -> PB1
- U11 pad 6: /STM32L432KCUx/PA0 -> PA0
- U11 pad 7: /STM32L432KCUx/PA1 -> PA1
- U2 pad 1: unconnected-(U10-VDD-Pad1) -> +5V
- U2 pad 2: unconnected-(U10-VOUT-Pad2) -> PB1
- U2 pad 3: unconnected-(U10-GND-Pad3) -> GND
Routing:
- net /LM66200_1/VIN1: track 4.59 -> 20.7 mm
- net /Reverse_Polarity/UVLO_IN: track 0.00 -> 15.8 mm
- net Net-(D1-A): track 0.00 -> 5.15 mm
- net CELL_1+: track 2.74 -> 0.00 mm
- net (no net): track 0.00 -> 2.74 mm
- net Net-(LED7-A): track 0.00 -> 1.54 mm

Commit message: exported STEP
Parts:
- moved D1 138.0 mm to (34.4, 13.2)
- moved LED7 138.0 mm to (40.0, 3.81)
- moved Q5 138.0 mm to (35.2, 8.38)
- moved R26 138.0 mm to (37.0, 3.81)
- moved R27 138.0 mm to (38.5, 13.2)
- moved C10 107.0 mm to (50.5, 41.7)
- moved C11 107.0 mm to (50.5, 43.6)
- moved C12 107.0 mm to (50.5, 45.6)
- moved C7 107.0 mm to (50.5, 35.7)
- moved C8 107.0 mm to (50.5, 37.7)
- moved C9 107.0 mm to (50.5, 39.7)
- moved R21 107.0 mm to (64.2, 35.8)
- moved R22 107.0 mm to (64.2, 37.7)
- moved R23 107.0 mm to (64.2, 39.7)
- moved U1 44.1 mm to (97.0, 72.9)
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Routing:
- net (no net): track 2.74 -> 0.00 mm

Commit message: started proper layout
Parts:
- removed BT2: Battery_Cell, Rocketry_Manual:BAT_1121
- removed C10: 10n, Capacitor_SMD:C_0402_1005Metric
- removed C11: 100n, Capacitor_SMD:C_0402_1005Metric
- removed C12: 4.7u, Capacitor_SMD:C_0402_1005Metric
- removed the J2 at (93.7, 28.7)
- removed R23: 5.1K, Resistor_SMD:R_0402_1005Metric
- removed USB1: TYPE-C 14P LTH10.0, Rocketry_Easyeda:TYPE-C-SMD_918-468K2029Y50001
- added C20: 10uF 0603, Rocketry_Easyeda:C0603, F.Cu at (56.7, 50.6)
- added C21: 10uF 0603, Rocketry_Easyeda:C0603, F.Cu at (58.5, 50.6)
- added C22: 10uF 0603, Rocketry_Easyeda:C0603, F.Cu at (56.7, 53.7)
- added C23: 100nF 0603, Rocketry_Easyeda:C0603, F.Cu at (62.0, 57.0)
- added C24: 22uF 0805, Rocketry_Easyeda:C0805, F.Cu at (68.4, 54.2)
- added C25: 22uF 0805, Rocketry_Easyeda:C0805, F.Cu at (70.4, 54.2)
- added C26: 22uF 0805, Rocketry_Easyeda:C0805, F.Cu at (72.5, 54.2)
- added C27: 4.7uF 0603, Rocketry_Easyeda:C0603, F.Cu at (89.7, 70.5)
- added C28: 100nF 0603, Rocketry_Easyeda:C0603, F.Cu at (80.5, 68.1)
- added C29: 10nF 0603, Rocketry_Easyeda:C0603, F.Cu at (80.5, 69.8)
- added J4: 1053091102, Rocketry_Manual:CON_1053091102, F.Cu at (114.3, 55.7)
- added LED7: 0805G (Green), Rocketry_Easyeda:LED0805-R-RD, F.Cu at (59.5, 58.0)
- added R32: 10k 0603, Rocketry_Easyeda:R0603, F.Cu at (58.5, 53.7)
- added R33: 680k 0603, Rocketry_Easyeda:R0603, F.Cu at (64.1, 53.7)
- added R34: 130k 0603, Rocketry_Easyeda:R0603, F.Cu at (64.1, 56.8)
- added R35: 330R 0603, Rocketry_Easyeda:R0603, F.Cu at (65.9, 58.0)
- added R36: 100k 0603, Rocketry_Easyeda:R0603, F.Cu at (104.4, 47.0)
- added R37: 100k 0603, Rocketry_Easyeda:R0603, F.Cu at (104.4, 64.8)
- added R38: 100k 0603, Rocketry_Easyeda:R0603, F.Cu at (104.4, 55.9)
- added R39: 5.1k 0603, Rocketry_Easyeda:R0603, F.Cu at (6.85, 46.2)
- added U16: 1.5uF 2.9A, Rocketry_Easyeda:IND-SMD_L2.5-W2.0_MEKK2520TR47M, F.Cu at (61.3, 50.2)
- added U17: TPS63070RNMR, Rocketry_Easyeda:VQFN-HR-15_L3.0-W2.5-P0.50-BL_TPS63070RNMR, F.Cu at (61.3, 53.7)
- BT1: value Battery_Cell -> 2P 21700 Cell Holder; footprint Rocketry_Manual:BAT_1121 -> Rocketry_Manual:PA21700x2-THM_Parallel
- C7: value 4.7u -> 100nF 0603; footprint Capacitor_SMD:C_0402_1005Metric -> Rocketry_Easyeda:C0603
- C8: value 100n -> 100nF 0603; footprint Capacitor_SMD:C_0402_1005Metric -> Rocketry_Easyeda:C0603
- C9: value 100n -> 4.7uF 0603; footprint Capacitor_SMD:C_0402_1005Metric -> Rocketry_Easyeda:C0603
- J1, J3: value Molex_Microfit -> 1053091102; footprint Rocketry_Manual:1054301102 -> Rocketry_Manual:CON_1053091102
- R21, R22: value 5.1K -> 5.1k 0603; footprint Resistor_SMD:R_0402_1005Metric -> Rocketry_Easyeda:R0603
- moved R18 131.2 mm to (46.5, 50.2), turned to -90 degrees
- moved U8 130.5 mm to (44.5, 50.0), turned to -90 degrees
- moved R19 124.7 mm to (46.5, 46.7), turned to -90 degrees
- moved U9 124.1 mm to (44.3, 46.7), turned to -90 degrees
- moved R17 91.0 mm to (37.6, 41.9)
- moved U7 91.0 mm to (37.4, 44.5)
- moved BT1 68.0 mm to (27.9, 125.9), turned to 90 degrees
- moved U2 67.3 mm to (114.1, 98.2), turned to 0 degrees
- moved J2 66.6 mm to (65.8, 69.1)
- moved C18 62.6 mm to (70.4, 39.0)
- moved C17 62.6 mm to (68.4, 39.0)
- moved C19 62.6 mm to (72.5, 39.0)
- moved C16 59.5 mm to (62.0, 41.9), turned to 90 degrees
- moved C15 58.9 mm to (56.7, 38.6)
- moved R28 58.9 mm to (58.5, 38.6)
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- renumbered J4 to J2, LED7 to LED5
Connections:
- C1 pad 1: /BQ29700_1/CELL- -> CELL_1-
- C2 pad 1: /BQ29700_2/CELL- -> CELL_2-
- C9 pad 2: +3.3V -> /STM32L432KCUx/+3V3A
- J1 pad 1: unconnected-(J1-Pin_1-Pad1) -> /LM66200_4/VOUT
- J1 pad 2: unconnected-(J1-Pin_2-Pad2) -> GND
- J3 pad 1: unconnected-(J3-Pin_1-Pad1) -> /LM66200_5/VOUT
- J3 pad 2: unconnected-(J3-Pin_2-Pad2) -> GND
- Q2 pad 2: /BQ29700_1/CELL- -> CELL_1-
- Q4 pad 2: /BQ29700_2/CELL- -> CELL_2-
- Q5 pad 2: /Reverse_Polarity/UVLO_IN -> USB_+5V
- R11 pad 1: /BQ29700_2/CELL- -> CELL_2-
- R20 pad 2: /LM66200_4/VIN1 -> +5V
- R21 pad 1: Net-(USB2-CC1) -> Net-(USB2-CC2)
- R22 pad 1: Net-(USB2-CC2) -> GND
- R22 pad 2: GND -> Net-(U11-PH3)
- R24 pad 2: /LM66200_5/VIN1 -> +5V
- R25 pad 2: /LM66200_6/VIN1 -> +5V
- R26 pad 2: /Reverse_Polarity/UVLO_IN -> USB_+5V
- R7 pad 1: /BQ29700_1/CELL- -> CELL_1-
- U1 pad 1: +5V -> +3.3V
- U10 pad 3: /LM66200_4/VIN1 -> +5V
- U10 pad 6: /LM66200_4/VIN1 -> +5V
- U12 pad 3: /LM66200_5/VIN1 -> +5V
- U12 pad 6: /LM66200_5/VIN1 -> +5V
- U13 pad 3: /LM66200_6/VIN1 -> +5V
- U13 pad 6: /LM66200_6/VIN1 -> +5V
- U2 pad 1: +5V -> +3.3V
- U3 pad 4: /BQ29700_1/CELL- -> CELL_1-
- U4 pad 4: /BQ29700_2/CELL- -> CELL_2-
- U7 pad 6: /LM66200_1/VIN2 -> /LM66200_1/VIN1
- USB2 pad 11: /STM32L432KCUx/VBUS -> USB_+5V
- USB2 pad 2: /STM32L432KCUx/VBUS -> USB_+5V
Routing:
- net CELL_2-: track 0.00 -> 78.9 mm
- net CELL_1-: track 0.00 -> 74.3 mm
- net CELL_1+: track 0.00 -> 70.3 mm
- net CELL_2+: track 0.00 -> 66.2 mm
- net USB_+5V: track 0.00 -> 23.5 mm
- net /Reverse_Polarity/UVLO_IN: track 15.8 -> 0.00 mm
- net Net-(LED3-C): track 0.00 -> 8.81 mm
- net Net-(LED7-A): track 0.00 -> 6.47 mm
- net /STM32L432KCUx/DN: track 0.00 -> 4.42 mm
- net /STM32L432KCUx/DP: track 0.00 -> 4.42 mm
- net /LM66200_1/VOUT: track 3.58 -> 0.00 mm
- net Net-(U17-EN): track 0.00 -> 3.25 mm
- net Net-(U17-FB): track 0.00 -> 2.99 mm
- net Net-(LED7-K): track 0.00 -> 2.89 mm
- net /LM66200_1/VIN2: track 2.42 -> 0.00 mm
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- added copper zone on F.Cu, net +5V
- added copper zone on F.Cu, net /LM66200_1/VOUT
- added copper zone on F.Cu, net /LM66200_2/VOUT
- added copper zone on F.Cu, net /LM66200_4/VOUT
- added copper zone on F.Cu, net /LM66200_5/VOUT
- added copper zone on F.Cu, net /LM66200_6/VOUT
- added copper zone on F.Cu, net CELL_1+
- added copper zone on F.Cu, net CELL_1-
- added copper zone on F.Cu, net CELL_2+
- added copper zone on F.Cu, net CELL_2-
- added copper zone on F.Cu, net Net-(Q1-D)
- added copper zone on F.Cu, net Net-(Q1-G)
- added copper zone on F.Cu, net Net-(Q2-G)
- added copper zone on F.Cu, net Net-(Q3-D)
- added copper zone on F.Cu, net Net-(Q3-G)
- added copper zone on F.Cu, net Net-(Q4-G)
- added copper zone on F.Cu, net Net-(U15-L1)
- added copper zone on F.Cu, net Net-(U15-L2)
- added copper zone on F.Cu, net Net-(U17-L1)
- added copper zone on F.Cu, net Net-(U17-L2)
- added copper zone on F.Cu, net Net-(U3-BAT)
- added copper zone on F.Cu, net Net-(U3-V-)
- added copper zone on F.Cu, net Net-(U4-BAT)
- added copper zone on F.Cu, net Net-(U4-V-)
- added copper zone on F.Cu, net Net-(U5-PROG)
- added copper zone on F.Cu, net Net-(U6-PROG)
Other:
- board size 199.4 x 114.2 mm -> 100 x 100 mm

Commit message: v0.1 sent to JLCPCB
Parts:
- removed the J2 at (65.8, 69.1)
- added C27: 100nF 0603, Rocketry_Easyeda:C0603, F.Cu at (104.1, 35.6)
- added C28: 100nF 0603, Rocketry_Easyeda:C0603, F.Cu at (104.1, 44.7)
- added C29: 100nF 0603, Rocketry_Easyeda:C0603, F.Cu at (104.4, 53.3)
- added C30: 10uF 0603, Rocketry_Easyeda:C0603, F.Cu at (56.6, 64.8)
- added C31: 10uF 0603, Rocketry_Easyeda:C0603, F.Cu at (58.4, 64.8)
- added C32: 10uF 0603, Rocketry_Easyeda:C0603, F.Cu at (56.6, 67.9)
- added C33: 100nF 0603, Rocketry_Easyeda:C0603, F.Cu at (62.0, 71.2)
- added C34: 22uF 0805, Rocketry_Easyeda:C0805, F.Cu at (68.3, 68.3)
- added C35: 22uF 0805, Rocketry_Easyeda:C0805, F.Cu at (70.3, 68.3)
- added C36: 22uF 0805, Rocketry_Easyeda:C0805, F.Cu at (72.4, 68.3)
- added C37: 10uF 0603, Rocketry_Easyeda:C0603, F.Cu at (82.4, 48.9)
- added C38: 10uF 0603, Rocketry_Easyeda:C0603, F.Cu at (82.4, 50.7)
- added C39: 10uF 0603, Rocketry_Easyeda:C0603, F.Cu at (82.4, 52.5)
- added C40: 10uF 0603, Rocketry_Easyeda:C0603, F.Cu at (82.5, 56.0)
- added C41: 10uF 0603, Rocketry_Easyeda:C0603, F.Cu at (82.4, 54.2)
- added C42: 10uF 0603, Rocketry_Easyeda:C0603, F.Cu at (85.7, 48.9)
- added C43: 10uF 0603, Rocketry_Easyeda:C0603, F.Cu at (85.7, 50.7)
- added C44: 10uF 0603, Rocketry_Easyeda:C0603, F.Cu at (85.7, 52.5)
- added C45: 10uF 0603, Rocketry_Easyeda:C0603, F.Cu at (85.7, 54.2)
- added C46: 10uF 0603, Rocketry_Easyeda:C0603, F.Cu at (85.7, 56.0)
- added G***: LOGO, Rocketry_Manual:RocketryLogo, B.Cu at (95.0, 94.0)
- added J4: Conn_01x05_Pin, Connector_PinHeader_2.54mm:PinHeader_1x05_P2.54mm_Vertical, F.Cu at (80.4, 29.7)
- added LED8: 0805G (Green), Rocketry_Easyeda:LED0805-R-RD, F.Cu at (59.2, 72.1)
- added R39: 10k 0603, Rocketry_Easyeda:R0603, F.Cu at (58.4, 67.9)
- added R40: 300k 0603, Rocketry_Easyeda:R0603, F.Cu at (64.0, 67.9)
- added R41: 33k 0603, Rocketry_Easyeda:R0603, F.Cu at (65.8, 69.2)
- added R42: 33k 0603, Rocketry_Easyeda:R0603, F.Cu at (64.0, 71.0)
- added R43: 330R 0603, Rocketry_Easyeda:R0603, F.Cu at (66.5, 72.5)
- added TP1: TestPoint, TestPoint:TestPoint_Pad_1.0x1.0mm, F.Cu at (41.1, 50.8)
- added TP10: TestPoint, TestPoint:TestPoint_Pad_1.0x1.0mm, F.Cu at (74.5, 40.1)
- added TP2: TestPoint, TestPoint:TestPoint_Pad_1.0x1.0mm, F.Cu at (47.5, 50.8)
- added TP3: TestPoint, TestPoint:TestPoint_Pad_1.0x1.0mm, F.Cu at (85.3, 75.2)
- added TP4: TestPoint, TestPoint:TestPoint_Pad_1.0x1.0mm, F.Cu at (88.6, 75.2)
- added TP5: TestPoint, TestPoint:TestPoint_Pad_1.0x1.0mm, F.Cu at (76.2, 53.1)
- added TP6: TestPoint, TestPoint:TestPoint_Pad_1.0x1.0mm, F.Cu at (76.2, 37.8)
- added TP7: TestPoint, TestPoint:TestPoint_Pad_1.0x1.0mm, F.Cu at (74.4, 67.3)
- added TP8: TestPoint, TestPoint:TestPoint_Pad_1.0x1.0mm, F.Cu at (72.9, 71.6)
- added TP9: TestPoint, TestPoint:TestPoint_Pad_1.0x1.0mm, F.Cu at (33.5, 48.8)
- added U18: 20m 1206, Rocketry_Easyeda:R1206, F.Cu at (105.7, 38.4)
- added U19: INA199A1DCKR, Rocketry_Easyeda:SC-70-6_L2.2-W1.3-P0.65-LS2.1-BR, F.Cu at (106.4, 35.6)
- added U20: 20m 1206, Rocketry_Easyeda:R1206, F.Cu at (105.7, 47.5)
- added U21: INA199A1DCKR, Rocketry_Easyeda:SC-70-6_L2.2-W1.3-P0.65-LS2.1-BR, F.Cu at (106.4, 44.7)
- added U22: 20m 1206, Rocketry_Easyeda:R1206, F.Cu at (105.9, 56.1)
- added U23: INA199A1DCKR, Rocketry_Easyeda:SC-70-6_L2.2-W1.3-P0.65-LS2.1-BR, F.Cu at (106.7, 53.3)
- added U24: 1.5uF 2.9A, Rocketry_Easyeda:IND-SMD_L2.5-W2.0_MEKK2520TR47M, F.Cu at (61.2, 64.3)
- added U25: TPS63070RNMR, Rocketry_Easyeda:VQFN-HR-15_L3.0-W2.5-P0.50-BL_TPS63070RNMR, F.Cu at (61.2, 67.8)
- added U26: 1.5uF 2.9A, Rocketry_Easyeda:IND-SMD_L2.5-W2.0_MEKK2520TR47M, F.Cu at (84.4, 46.6)
- moved R26 84.1 mm to (89.0, 61.5), turned to -90 degrees
- moved U1 55.4 mm to (59.0, 102.0), turned to 90 degrees
- moved R2 47.0 mm to (46.7, 63.2), turned to 180 degrees
- moved R1 43.1 mm to (43.7, 63.2), turned to 180 degrees
- moved R4 42.1 mm to (47.0, 75.4), turned to 180 degrees
- moved R24 42.1 mm to (48.0, 37.6)
- moved R3 38.2 mm to (43.9, 75.4), turned to 180 degrees
- moved R25 37.5 mm to (44.2, 38.5), turned to -90 degrees
- moved U2 35.3 mm to (79.0, 102.0), turned to 90 degrees
- moved R27 18.7 mm to (98.9, 50.2)
- moved R6 18.7 mm to (96.8, 47.6)
- moved U12 18.7 mm to (98.8, 47.6)
- moved J2 17.1 mm to (112.4, 47.5)
- moved R5 11.3 mm to (96.8, 38.6)
- moved U10 11.3 mm to (98.8, 38.6)
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- renumbered C29 to C10, C28 to C11, C9 to C12, C27 to C7, C7 to C8, C8 to C9, J3 to J2, J4 to J3, R7 to R10, R8 to R11, R9 to R12, R10 to R13, R11 to R14, R12 to R15, R13 to R16, R14 to R17, R15 to R18, R16 to R19, R17 to R20, R18 to R21, R19 to R22, R20 to R23, R39 to R24, R21 to R25, R22 to R26, R24 to R27, R25 to R28, R26 to R29, R27 to R30, R28 to R31, R29 to R32, R30 to R33, R31 to R34, R32 to R35, R33 to R36, R34 to R37, R35 to R38, R36 to R5, R37 to R6, R38 to R7, R5 to R8, R6 to R9, USB2 to USB1
Connections:
- J1 pad 1: /LM66200_4/VOUT -> /INA199_1/IN-
- J2 pad 1: /LM66200_5/VOUT -> /INA199_2/IN-
- J3 pad 1: /LM66200_6/VOUT -> /INA199_3/IN-
- R23 pad 2: +5V -> +9V
- R28 pad 2: +5V -> +3.3V
- U10 pad 2: /LM66200_4/VOUT -> /INA199_1/IN+
- U10 pad 3: +5V -> +9V
- U10 pad 6: +5V -> +9V
- U10 pad 7: /LM66200_4/VOUT -> /INA199_1/IN+
- U11 pad 10: /STM32L432KCUx/PA4 -> INA199_3
- U11 pad 8: /STM32L432KCUx/PA2 -> INA199_1
- U11 pad 9: /STM32L432KCUx/PA3 -> INA199_2
- U12 pad 2: /LM66200_5/VOUT -> /INA199_2/IN+
- U12 pad 7: /LM66200_5/VOUT -> /INA199_2/IN+
- U13 pad 2: /LM66200_6/VOUT -> /INA199_3/IN+
- U13 pad 3: +5V -> +3.3V
- U13 pad 6: +5V -> +3.3V
- U13 pad 7: /LM66200_6/VOUT -> /INA199_3/IN+
Routing:
- net GND: track 5.08 -> 157.7 mm, vias 4 -> 245
- net +3.3V: track 0.00 -> 80.8 mm, vias 0 -> 24
- net CELL_2-: track 78.9 -> 0.00 mm, vias 0 -> 5
- net CELL_1-: track 74.3 -> 0.00 mm, vias 0 -> 6
- net /STM32L432KCUx/DN: track 4.42 -> 75.0 mm, vias 0 -> 2
- net /STM32L432KCUx/DP: track 4.42 -> 74.1 mm, vias 0 -> 2
- net CELL_1+: track 70.3 -> 11.8 mm, vias 0 -> 16
- net CELL_2+: track 66.2 -> 10.7 mm, vias 0 -> 15
- net INA199_1: track 0.00 -> 51.9 mm, vias 0 -> 3
- net PA0: track 0.00 -> 51.3 mm, vias 0 -> 2
- net PB0: track 0.00 -> 47.0 mm, vias 0 -> 1
- net PA1: track 0.00 -> 45.7 mm, vias 0 -> 2
- net INA199_2: track 0.00 -> 44.9 mm, vias 0 -> 3
- net /STM32L432KCUx/nRST: track 0.00 -> 43.2 mm, vias 0 -> 4
- net ~{MCU_LS_1}: track 1.34 -> 44.1 mm, vias 0 -> 2
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- added copper zone on F.Cu, net +3.3V
- added copper zone on In1.Cu, net +3.3V
- added copper zone on In2.Cu, net +5V
- added copper zone on F.Cu, net +9V
- added copper zone on F.Cu, net /INA199_1/IN+
- added copper zone on F.Cu, net /INA199_1/IN-
- added copper zone on F.Cu, net /INA199_2/IN+
- added copper zone on F.Cu, net /INA199_2/IN-
- added copper zone on F.Cu, net /INA199_3/IN+
- added copper zone on F.Cu, net /INA199_3/IN-
- added copper zone on F.Cu, net /STM32L432KCUx/+3V3A
- added copper zone on B.Cu, net CELL_1+
- added copper zone on B.Cu, net CELL_1-
- added copper zone on B.Cu, net CELL_2+
- added copper zone on In1.Cu, net CELL_2+
- added copper zone on B.Cu, net CELL_2-
- added copper zone on In1.Cu, net GND
- added copper zone on In2.Cu, net GND
- added copper zone on F.Cu, net Net-(D1-A)
- added copper zone on F.Cu, net Net-(U25-L1)
- added copper zone on F.Cu, net Net-(U25-L2)
- added copper zone on F.Cu, net USB_+5V
- removed copper zone on F.Cu, net /LM66200_4/VOUT
- removed copper zone on F.Cu, net /LM66200_5/VOUT
- removed copper zone on F.Cu, net /LM66200_6/VOUT
Other:
- board text added: "+3.3V"
- board text added: "3.3V"
- board text added: "5V"
- board text added: "9V"
- board text added: "EPS V0.1 Test Board"
- board text added: "GND"
- board text added: "McMaster Rocketry"
- board text added: "SWCLK"
- board text added: "SWDIO"
- board text added: "nRST"
