File: v2/blocks/LM66200_4.kicad_sch (KiCad schematic)
At the start: 2 parts, among them U8 C3235556 (M66200DRLR)

Commit message: preliminary layout
Parts:
- renumbered R23 to R22, U8 to U7
Changed lines of the file:
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@@
 		(on_board yes)
 		(dnp no)
-		(property "Reference" "R23"
+		(property "Reference" "R22"
 			(at 123.952 48.26 90)
 			(effects
@@
 			(project "EPSv1"
 				(path "/61d36b12-c329-4dd2-b08b-b63678fc7b25/48ef5cbc-bda3-4680-a2aa-3beff134f7df"
-					(reference "R23")
+					(reference "R22")
 					(unit 1)
 				)
@@
 		(dnp no)
 		(fields_autoplaced yes)
-		(property "Reference" "U8"
+		(property "Reference" "U7"
 			(at 101.6 44.45 0)
 			(effects
@@
 			(project "EPSv1"
 				(path "/61d36b12-c329-4dd2-b08b-b63678fc7b25/48ef5cbc-bda3-4680-a2aa-3beff134f7df"
-					(reference "U8")
+					(reference "U7")
 					(unit 1)
 				)
