File: v2/blocks/LM66200_5.kicad_sch (KiCad schematic)
At the start: 2 parts, among them U10 C3235556 (M66200DRLR)

Commit message: preliminary layout
Parts:
- renumbered R27 to R24, U10 to U9
Changed lines of the file:
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@@
 		(dnp no)
 		(fields_autoplaced yes)
-		(property "Reference" "U10"
+		(property "Reference" "U9"
 			(at 101.6 44.45 0)
 			(effects
@@
 			(project "EPSv1"
 				(path "/61d36b12-c329-4dd2-b08b-b63678fc7b25/3730cabe-0fc6-42a7-882b-11af5299f645"
-					(reference "U10")
+					(reference "U9")
 					(unit 1)
 				)
@@
 		(on_board yes)
 		(dnp no)
-		(property "Reference" "R27"
+		(property "Reference" "R24"
 			(at 123.952 48.26 90)
 			(effects
@@
 			(project "EPSv1"
 				(path "/61d36b12-c329-4dd2-b08b-b63678fc7b25/3730cabe-0fc6-42a7-882b-11af5299f645"
-					(reference "R27")
+					(reference "R24")
 					(unit 1)
 				)
