File: v2/blocks/LM66200_6.kicad_sch (KiCad schematic)
At the start: 2 parts, among them U11 C3235556 (M66200DRLR)

Commit message: preliminary layout
Parts:
- renumbered R28 to R25, U11 to U10
Changed lines of the file:
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@@
 		(on_board yes)
 		(dnp no)
-		(property "Reference" "R28"
+		(property "Reference" "R25"
 			(at 123.952 48.26 90)
 			(effects
@@
 			(project "EPSv1"
 				(path "/61d36b12-c329-4dd2-b08b-b63678fc7b25/1de4be1f-e3cc-4463-a609-d6709bdbcf35"
-					(reference "R28")
+					(reference "R25")
 					(unit 1)
 				)
@@
 		(dnp no)
 		(fields_autoplaced yes)
-		(property "Reference" "U11"
+		(property "Reference" "U10"
 			(at 101.6 44.45 0)
 			(effects
@@
 			(project "EPSv1"
 				(path "/61d36b12-c329-4dd2-b08b-b63678fc7b25/1de4be1f-e3cc-4463-a609-d6709bdbcf35"
-					(reference "U11")
+					(reference "U10")
 					(unit 1)
 				)
