File: v2/blocks/BQ29700_1.kicad_sch (KiCad schematic)
At the start: 8 parts, among them Q1 AO3400A, Q2 AO3400A, U1 BQ29700DSER

Commit message: battery charging routing
Parts:
- renumbered C11 to C3
Changed lines of the file:
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@@
 		(dnp no)
 		(fields_autoplaced yes)
-		(property "Reference" "C11"
+		(property "Reference" "C3"
 			(at 128.27 62.2299 90)
 			(effects
@@
 			(project "EPSv2"
 				(path "/61d36b12-c329-4dd2-b08b-b63678fc7b25/b8a60f44-eeb8-489a-a794-4b296827b74d"
-					(reference "C11")
+					(reference "C3")
 					(unit 1)
 				)

Commit message: routing done
Parts:
- renumbered R8 to R5, R9 to R6, R10 to R7, R11 to R8
Changed lines of the file:
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@@
 		(dnp no)
 		(fields_autoplaced yes)
-		(property "Reference" "R11"
+		(property "Reference" "R8"
 			(at 127 52.0699 90)
 			(effects
@@
 			(project "EPSv2"
 				(path "/61d36b12-c329-4dd2-b08b-b63678fc7b25/b8a60f44-eeb8-489a-a794-4b296827b74d"
-					(reference "R11")
+					(reference "R8")
 					(unit 1)
 				)
@@
 		(on_board yes)
 		(dnp no)
-		(property "Reference" "R9"
+		(property "Reference" "R6"
 			(at 53.34 73.6599 90)
 			(effects
@@
 			(project "EPSv2"
 				(path "/61d36b12-c329-4dd2-b08b-b63678fc7b25/b8a60f44-eeb8-489a-a794-4b296827b74d"
-					(reference "R9")
+					(reference "R6")
 					(unit 1)
 				)
@@
 		(on_board yes)
 		(dnp no)
-		(property "Reference" "R8"
+		(property "Reference" "R5"
 			(at 40.64 64.7699 90)
 			(effects
@@
 			(project "EPSv2"
 				(path "/61d36b12-c329-4dd2-b08b-b63678fc7b25/b8a60f44-eeb8-489a-a794-4b296827b74d"
-					(reference "R8")
+					(reference "R5")
 					(unit 1)
 				)
@@
 		(dnp no)
 		(fields_autoplaced yes)
-		(property "Reference" "R10"
+		(property "Reference" "R7"
 			(at 82.55 73.6599 90)
 			(effects
@@
 			(project "EPSv2"
 				(path "/61d36b12-c329-4dd2-b08b-b63678fc7b25/b8a60f44-eeb8-489a-a794-4b296827b74d"
-					(reference "R10")
-					(unit 1)
-				)
+					(reference "R7")
+					(unit 1)
+				)

Commit message: can transceiver and battery reverse polarity bypass
Parts:
- renumbered R5 to R6, R6 to R7, R7 to R8, R8 to R9
Changed lines of the file:
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@@
 		(shape bidirectional)
 		(at 38.1 41.91 180)
+		(fields_autoplaced yes)
 		(effects
 			(font
@@
 		(shape bidirectional)
 		(at 146.05 41.91 0)
+		(fields_autoplaced yes)
 		(effects
 			(font
@@
 		(shape bidirectional)
 		(at 38.1 80.01 180)
+		(fields_autoplaced yes)
 		(effects
 			(font
@@
 		(shape bidirectional)
 		(at 146.05 80.01 0)
+		(fields_autoplaced yes)
 		(effects
 			(font
@@
 		(dnp no)
 		(fields_autoplaced yes)
-		(property "Reference" "R8"
+		(property "Reference" "R9"
 			(at 127 52.0699 90)
 			(effects
@@
 			(project "EPSv2"
 				(path "/61d36b12-c329-4dd2-b08b-b63678fc7b25/b8a60f44-eeb8-489a-a794-4b296827b74d"
-					(reference "R8")
+					(reference "R9")
 					(unit 1)
 				)
@@
 		(on_board yes)
 		(dnp no)
-		(property "Reference" "R6"
+		(property "Reference" "R7"
 			(at 53.34 73.6599 90)
 			(effects
@@
 			(project "EPSv2"
 				(path "/61d36b12-c329-4dd2-b08b-b63678fc7b25/b8a60f44-eeb8-489a-a794-4b296827b74d"
-					(reference "R6")
+					(reference "R7")
 					(unit 1)
 				)
@@
 		(on_board yes)
 		(dnp no)
-		(property "Reference" "R5"
+		(property "Reference" "R6"
 			(at 40.64 64.7699 90)
 			(effects
@@
 			(project "EPSv2"
 				(path "/61d36b12-c329-4dd2-b08b-b63678fc7b25/b8a60f44-eeb8-489a-a794-4b296827b74d"
-					(reference "R5")
+					(reference "R6")
 					(unit 1)
 				)
@@
 		(dnp no)
 		(fields_autoplaced yes)
-		(property "Reference" "R7"
+		(property "Reference" "R8"
 			(at 82.55 73.6599 90)
 			(effects
@@
 			(project "EPSv2"
 				(path "/61d36b12-c329-4dd2-b08b-b63678fc7b25/b8a60f44-eeb8-489a-a794-4b296827b74d"
-					(reference "R7")
-					(unit 1)
-				)
+					(reference "R8")
+					(unit 1)
+				)
