File: v2/blocks/LM66200_2.kicad_sch (KiCad schematic)
At the start: 2 parts, among them U6 C3235556 (M66200DRLR)

Commit message: preliminary layout
Parts:
- renumbered R21 to R20, U6 to U5
Changed lines of the file:
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@@
 		(on_board yes)
 		(dnp no)
-		(property "Reference" "R21"
+		(property "Reference" "R20"
 			(at 123.952 48.26 90)
 			(effects
@@
 			(project "EPSv1"
 				(path "/61d36b12-c329-4dd2-b08b-b63678fc7b25/ba3c3b19-82c2-46ed-8aa1-9c2c518efa44"
-					(reference "R21")
+					(reference "R20")
 					(unit 1)
 				)
@@
 		(dnp no)
 		(fields_autoplaced yes)
-		(property "Reference" "U6"
+		(property "Reference" "U5"
 			(at 101.6 44.45 0)
 			(effects
@@
 			(project "EPSv1"
 				(path "/61d36b12-c329-4dd2-b08b-b63678fc7b25/ba3c3b19-82c2-46ed-8aa1-9c2c518efa44"
-					(reference "U6")
+					(reference "U5")
 					(unit 1)
 				)

Commit message: routing done
Parts:
- renumbered R20 to R24, U5 to U6
Changed lines of the file:
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@@
 		(on_board yes)
 		(dnp no)
-		(property "Reference" "R20"
+		(property "Reference" "R24"
 			(at 123.952 48.26 90)
 			(effects
@@
 			(project "EPSv1"
 				(path "/61d36b12-c329-4dd2-b08b-b63678fc7b25/ba3c3b19-82c2-46ed-8aa1-9c2c518efa44"
-					(reference "R20")
+					(reference "R24")
 					(unit 1)
 				)
@@
 		(dnp no)
 		(fields_autoplaced yes)
-		(property "Reference" "U5"
+		(property "Reference" "U6"
 			(at 101.6 44.45 0)
 			(effects
@@
 			(project "EPSv1"
 				(path "/61d36b12-c329-4dd2-b08b-b63678fc7b25/ba3c3b19-82c2-46ed-8aa1-9c2c518efa44"
-					(reference "U5")
+					(reference "U6")
 					(unit 1)
 				)

Commit message: can transceiver and battery reverse polarity bypass
Parts:
- renumbered R24 to R25
Changed lines of the file:
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@@
 		(shape input)
 		(at 113.03 57.15 0)
+		(fields_autoplaced yes)
 		(effects
 			(font
@@
 		(shape input)
 		(at 83.82 59.69 180)
+		(fields_autoplaced yes)
 		(effects
 			(font
@@
 		(shape output)
 		(at 124.46 54.61 0)
+		(fields_autoplaced yes)
 		(effects
 			(font
@@
 		(shape input)
 		(at 113.03 59.69 0)
+		(fields_autoplaced yes)
 		(effects
 			(font
@@
 		(shape input)
 		(at 83.82 57.15 180)
+		(fields_autoplaced yes)
 		(effects
 			(font
@@
 		(shape input)
 		(at 83.82 52.07 180)
+		(fields_autoplaced yes)
 		(effects
 			(font
@@
 		(shape input)
 		(at 120.65 39.37 180)
+		(fields_autoplaced yes)
 		(effects
 			(font
@@
 		(on_board yes)
 		(dnp no)
-		(property "Reference" "R24"
+		(property "Reference" "R25"
 			(at 123.952 48.26 90)
 			(effects
@@
 			(project "EPSv1"
 				(path "/61d36b12-c329-4dd2-b08b-b63678fc7b25/ba3c3b19-82c2-46ed-8aa1-9c2c518efa44"
-					(reference "R24")
+					(reference "R25")
 					(unit 1)
 				)
