File: v2/blocks/MCP73831_1.kicad_sch (KiCad schematic)
At the start: 6 parts, among them U3 MCP73831T-2ACI/OT

Commit message: battery charging routing
Parts:
- renumbered C13 to C5, C14 to C6
Changed lines of the file:
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@@
 		(on_board yes)
 		(dnp no)
-		(property "Reference" "C13"
+		(property "Reference" "C5"
 			(at 40.64 54.6099 90)
 			(effects
@@
 			(project "EPSv2"
 				(path "/61d36b12-c329-4dd2-b08b-b63678fc7b25/103c9400-3c4a-46fe-9b91-cdd5ca031b83"
-					(reference "C13")
+					(reference "C5")
 					(unit 1)
 				)
@@
 		(on_board yes)
 		(dnp no)
-		(property "Reference" "C14"
+		(property "Reference" "C6"
 			(at 151.13 66.0399 90)
 			(effects
@@
 			(project "EPSv2"
 				(path "/61d36b12-c329-4dd2-b08b-b63678fc7b25/103c9400-3c4a-46fe-9b91-cdd5ca031b83"
-					(reference "C14")
-					(unit 1)
-				)
+					(reference "C6")
+					(unit 1)
+				)

Commit message: routing done
Parts:
- renumbered R16 to R13, R17 to R14
Changed lines of the file:
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@@
 		(dnp no)
 		(fields_autoplaced yes)
-		(property "Reference" "R16"
+		(property "Reference" "R13"
 			(at 78.74 62.23 0)
 			(effects
@@
 			(project ""
 				(path "/61d36b12-c329-4dd2-b08b-b63678fc7b25/103c9400-3c4a-46fe-9b91-cdd5ca031b83"
-					(reference "R16")
+					(reference "R13")
 					(unit 1)
 				)
@@
 		(dnp no)
 		(fields_autoplaced yes)
-		(property "Reference" "R17"
+		(property "Reference" "R14"
 			(at 130.81 64.7699 90)
 			(effects
@@
 			(project "EPSv2"
 				(path "/61d36b12-c329-4dd2-b08b-b63678fc7b25/103c9400-3c4a-46fe-9b91-cdd5ca031b83"
-					(reference "R17")
+					(reference "R14")
 					(unit 1)
 				)

Commit message: can transceiver and battery reverse polarity bypass
Parts:
- renumbered R13 to R14, R14 to R15
Changed lines of the file:
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@@
 		(shape input)
 		(at 38.1 45.72 180)
+		(fields_autoplaced yes)
 		(effects
 			(font
@@
 		(shape input)
 		(at 124.46 85.09 270)
+		(fields_autoplaced yes)
 		(effects
 			(font
@@
 		(shape output)
 		(at 151.13 57.15 0)
+		(fields_autoplaced yes)
 		(effects
 			(font
@@
 		(dnp no)
 		(fields_autoplaced yes)
-		(property "Reference" "R13"
+		(property "Reference" "R14"
 			(at 78.74 62.23 0)
 			(effects
@@
 			(project ""
 				(path "/61d36b12-c329-4dd2-b08b-b63678fc7b25/103c9400-3c4a-46fe-9b91-cdd5ca031b83"
-					(reference "R13")
+					(reference "R14")
 					(unit 1)
 				)
@@
 		(dnp no)
 		(fields_autoplaced yes)
-		(property "Reference" "R14"
+		(property "Reference" "R15"
 			(at 130.81 64.7699 90)
 			(effects
@@
 			(project "EPSv2"
 				(path "/61d36b12-c329-4dd2-b08b-b63678fc7b25/103c9400-3c4a-46fe-9b91-cdd5ca031b83"
-					(reference "R14")
+					(reference "R15")
 					(unit 1)
 				)
