File: v2/blocks/STM32L432KCUx.kicad_sch (KiCad schematic)
At the start: 9 parts, among them J10 Conn_01x05_Pin, U9 STM32L432KCUx

Commit message: preliminary layout
Parts:
- renumbered R26 to R23, U9 to U8
Changed lines of the file:
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@@
 		(dnp no)
 		(fields_autoplaced yes)
-		(property "Reference" "R26"
+		(property "Reference" "R23"
 			(at 171.45 53.34 0)
 			(effects
@@
 			(project "EPSv2"
 				(path "/61d36b12-c329-4dd2-b08b-b63678fc7b25/cef003e9-4e09-46ce-a170-d9263c8f93eb"
-					(reference "R26")
+					(reference "R23")
 					(unit 1)
 				)
@@
 		(dnp no)
 		(fields_autoplaced yes)
-		(property "Reference" "U9"
+		(property "Reference" "U8"
 			(at 197.7741 100.33 0)
 			(effects
@@
 			(project "EPSv2"
 				(path "/61d36b12-c329-4dd2-b08b-b63678fc7b25/cef003e9-4e09-46ce-a170-d9263c8f93eb"
-					(reference "U9")
+					(reference "U8")
 					(unit 1)
 				)

Commit message: battery charging routing
Parts:
- renumbered C18 to C10, C19 to C11, C20 to C12, C21 to C13, C22 to C14, C17 to C9
Changed lines of the file:
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@@
 		(dnp no)
 		(fields_autoplaced yes)
-		(property "Reference" "C18"
+		(property "Reference" "C10"
 			(at 168.91 43.18 90)
 			(effects
@@
 			(project "EPSv2"
 				(path "/61d36b12-c329-4dd2-b08b-b63678fc7b25/cef003e9-4e09-46ce-a170-d9263c8f93eb"
-					(reference "C18")
+					(reference "C10")
 					(unit 1)
 				)
@@
 		(dnp no)
 		(fields_autoplaced yes)
-		(property "Reference" "C19"
+		(property "Reference" "C11"
 			(at 184.15 43.18 90)
 			(effects
@@
 			(project "EPSv2"
 				(path "/61d36b12-c329-4dd2-b08b-b63678fc7b25/cef003e9-4e09-46ce-a170-d9263c8f93eb"
-					(reference "C19")
+					(reference "C11")
 					(unit 1)
 				)
@@
 		(dnp no)
 		(fields_autoplaced yes)
-		(property "Reference" "C17"
+		(property "Reference" "C9"
 			(at 154.94 44.45 90)
 			(effects
@@
 			(project "EPSv2"
 				(path "/61d36b12-c329-4dd2-b08b-b63678fc7b25/cef003e9-4e09-46ce-a170-d9263c8f93eb"
-					(reference "C17")
+					(reference "C9")
 					(unit 1)
 				)
@@
 		(dnp no)
 		(fields_autoplaced yes)
-		(property "Reference" "C21"
+		(property "Reference" "C13"
 			(at 220.98 43.18 90)
 			(effects
@@
 			(project "EPSv2"
 				(path "/61d36b12-c329-4dd2-b08b-b63678fc7b25/cef003e9-4e09-46ce-a170-d9263c8f93eb"
-					(reference "C21")
+					(reference "C13")
 					(unit 1)
 				)
@@
 		(dnp no)
 		(fields_autoplaced yes)
-		(property "Reference" "C20"
+		(property "Reference" "C12"
 			(at 205.74 41.91 90)
 			(effects
@@
 			(project "EPSv2"
 				(path "/61d36b12-c329-4dd2-b08b-b63678fc7b25/cef003e9-4e09-46ce-a170-d9263c8f93eb"
-					(reference "C20")
+					(reference "C12")
 					(unit 1)
 				)
@@
 		(dnp no)
 		(fields_autoplaced yes)
-		(property "Reference" "C22"
+		(property "Reference" "C14"
 			(at 237.49 41.91 90)
 			(effects
@@
 			(project "EPSv2"
 				(path "/61d36b12-c329-4dd2-b08b-b63678fc7b25/cef003e9-4e09-46ce-a170-d9263c8f93eb"
-					(reference "C22")
-					(unit 1)
-				)
+					(reference "C14")
+					(unit 1)
+				)

Commit message: routing done
Parts:
- renumbered C9 to C11, C10 to C12, C11 to C13, C12 to C14, C13 to C15, C14 to C16, R23 to R26
Connections:
- net PB3: now reaches U8.26 (PB3)
- net PB4: now reaches U8.27 (PB4)
- net PB5: now reaches U8.28 (PB5)
- net PB6: now reaches U8.29 (PB6)
- net PB7: now reaches U8.30 (PB7)
Changed lines of the file:
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@@
+		)
+	)
+	(hierarchical_label "PB6"
+		(shape bidirectional)
+		(at 182.88 85.09 180)
+		(fields_autoplaced yes)
+		(effects
+			(font
+				(size 1.27 1.27)
+			)
+			(justify right)
 		)
 	)
@@
 		)
 	)
+	(hierarchical_label "PB4"
+		(shape bidirectional)
+		(at 182.88 80.01 180)
+		(fields_autoplaced yes)
+		(effects
+			(font
+				(size 1.27 1.27)
+			)
+			(justify right)
+		)
+	)
+	(hierarchical_label "PB5"
+		(shape bidirectional)
+		(at 182.88 82.55 180)
+		(fields_autoplaced yes)
+		(effects
+			(font
+				(size 1.27 1.27)
+			)
+			(justify right)
+		)
+	)
+	(hierarchical_label "PB7"
+		(shape bidirectional)
+		(at 182.88 87.63 180)
+		(fields_autoplaced yes)
+		(effects
+			(font
+				(size 1.27 1.27)
+			)
+			(justify right)
+		)
+	)
 	(hierarchical_label "PA0"
 		(shape bidirectional)
@@
 			)
 			(justify left)
+		)
+	)
+	(hierarchical_label "PB3"
+		(shape bidirectional)
+		(at 182.88 77.47 180)
+		(fields_autoplaced yes)
+		(effects
+			(font
+				(size 1.27 1.27)
+			)
+			(justify right)
 		)
 	)
@@
 		(dnp no)
 		(fields_autoplaced yes)
-		(property "Reference" "C10"
+		(property "Reference" "C12"
 			(at 168.91 43.18 90)
 			(effects
@@
 			(project "EPSv2"
 				(path "/61d36b12-c329-4dd2-b08b-b63678fc7b25/cef003e9-4e09-46ce-a170-d9263c8f93eb"
-					(reference "C10")
+					(reference "C12")
 					(unit 1)
 				)
@@
 		(dnp no)
 		(fields_autoplaced yes)
-		(property "Reference" "C11"
+		(property "Reference" "C13"
 			(at 184.15 43.18 90)
 			(effects
@@
 			(project "EPSv2"
 				(path "/61d36b12-c329-4dd2-b08b-b63678fc7b25/cef003e9-4e09-46ce-a170-d9263c8f93eb"
-					(reference "C11")
+					(reference "C13")
 					(unit 1)
 				)
@@
 		(dnp no)
 		(fields_autoplaced yes)
-		(property "Reference" "R23"
+		(property "Reference" "R26"
 			(at 171.45 53.34 0)
 			(effects
@@
 			(project "EPSv2"
 				(path "/61d36b12-c329-4dd2-b08b-b63678fc7b25/cef003e9-4e09-46ce-a170-d9263c8f93eb"
-					(reference "R23")
+					(reference "R26")
 					(unit 1)
 				)
@@
 		(dnp no)
 		(fields_autoplaced yes)
-		(property "Reference" "C9"
+		(property "Reference" "C11"
 			(at 154.94 44.45 90)
 			(effects
@@
 			(project "EPSv2"
 				(path "/61d36b12-c329-4dd2-b08b-b63678fc7b25/cef003e9-4e09-46ce-a170-d9263c8f93eb"
-					(reference "C9")
+					(reference "C11")
 					(unit 1)
 				)
@@
 		(dnp no)
 		(fields_autoplaced yes)
-		(property "Reference" "C13"
+		(property "Reference" "C15"
 			(at 220.98 43.18 90)
 			(effects
@@
 			(project "EPSv2"
 				(path "/61d36b12-c329-4dd2-b08b-b63678fc7b25/cef003e9-4e09-46ce-a170-d9263c8f93eb"
-					(reference "C13")
+					(reference "C15")
 					(unit 1)
 				)
@@
 		(dnp no)
 		(fields_autoplaced yes)
-		(property "Reference" "C12"
+		(property "Reference" "C14"
 			(at 205.74 41.91 90)
 			(effects
@@
 			(project "EPSv2"
 				(path "/61d36b12-c329-4dd2-b08b-b63678fc7b25/cef003e9-4e09-46ce-a170-d9263c8f93eb"
-					(reference "C12")
+					(reference "C14")
 					(unit 1)
 				)
@@
 		(dnp no)
 		(fields_autoplaced yes)
-		(property "Reference" "C14"
+		(property "Reference" "C16"
 			(at 237.49 41.91 90)
 			(effects
@@
 			(project "EPSv2"
 				(path "/61d36b12-c329-4dd2-b08b-b63678fc7b25/cef003e9-4e09-46ce-a170-d9263c8f93eb"
-					(reference "C14")
-					(unit 1)
-				)
+					(reference "C16")
+					(unit 1)
+				)

Commit message: CAN txrx
Connections:
- net PA11: now reaches U8.21 (PA11)
- net PA12: now reaches U8.22 (PA12)
- net PA8: no longer names the net of U8.18 (PA8)
Changed lines of the file:
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@@
 	(label "SWDIO"
 		(at 123.19 36.83 0)
-		(fields_autoplaced yes)
 		(effects
 			(font
@@
 	(label "GND"
 		(at 123.19 34.29 0)
-		(fields_autoplaced yes)
 		(effects
 			(font
@@
 	(label "GND"
 		(at 227.33 53.34 180)
-		(fields_autoplaced yes)
 		(effects
 			(font
@@
 	(label "SWDIO"
 		(at 208.28 87.63 0)
-		(fields_autoplaced yes)
 		(effects
 			(font
@@
 	(label "GND"
 		(at 195.58 104.14 180)
-		(fields_autoplaced yes)
 		(effects
 			(font
@@
 	(label "GND"
 		(at 157.48 54.61 180)
-		(fields_autoplaced yes)
 		(effects
 			(font
@@
 	(label "nRST"
 		(at 182.88 54.61 180)
-		(fields_autoplaced yes)
 		(effects
 			(font
@@
 	(label "SWDCLK"
 		(at 123.19 41.91 0)
-		(fields_autoplaced yes)
 		(effects
 			(font
@@
 	(label "GND"
 		(at 165.1 59.69 180)
-		(fields_autoplaced yes)
 		(effects
 			(font
@@
 	(label "nRST"
 		(at 123.19 31.75 0)
-		(fields_autoplaced yes)
 		(effects
 			(font
@@
 	(label "SWDCLK"
 		(at 208.28 90.17 0)
-		(fields_autoplaced yes)
 		(effects
 			(font
@@
 	(label "GND"
 		(at 55.88 30.48 0)
-		(fields_autoplaced yes)
 		(effects
 			(font
@@
 		(shape bidirectional)
 		(at 208.28 77.47 0)
-		(fields_autoplaced yes)
 		(effects
 			(font
@@
 		(shape bidirectional)
 		(at 182.88 72.39 180)
-		(fields_autoplaced yes)
 		(effects
 			(font
@@
 		(shape bidirectional)
 		(at 208.28 62.23 0)
-		(fields_autoplaced yes)
 		(effects
 			(font
@@
 		(shape bidirectional)
 		(at 182.88 74.93 180)
-		(fields_autoplaced yes)
 		(effects
 			(font
@@
 		(shape bidirectional)
 		(at 208.28 59.69 0)
-		(fields_autoplaced yes)
 		(effects
 			(font
@@
 		(shape bidirectional)
 		(at 208.28 64.77 0)
-		(fields_autoplaced yes)
 		(effects
 			(font
@@
 		(shape bidirectional)
 		(at 208.28 72.39 0)
-		(fields_autoplaced yes)
 		(effects
 			(font
@@
 		(shape input)
 		(at 142.24 35.56 180)
-		(fields_autoplaced yes)
-		(effects
-			(font
-				(size 1.27 1.27)
-			)
-			(justify right)
-		)
-	)
-	(hierarchical_label "PA8"
-		(shape bidirectional)
-		(at 208.28 74.93 0)
-		(fields_autoplaced yes)
-		(effects
-			(font
-				(size 1.27 1.27)
-			)
-			(justify left)
+		(effects
+			(font
+				(size 1.27 1.27)
+			)
+			(justify right)
 		)
 	)
@@
 		(shape bidirectional)
 		(at 182.88 85.09 180)
-		(fields_autoplaced yes)
 		(effects
 			(font
@@
 		(shape bidirectional)
 		(at 208.28 67.31 0)
-		(fields_autoplaced yes)
+		(effects
+			(font
+				(size 1.27 1.27)
+			)
+			(justify left)
+		)
+	)
+	(hierarchical_label "PA12"
+		(shape bidirectional)
+		(at 208.28 85.09 0)
 		(effects
 			(font
@@
 		(shape bidirectional)
 		(at 182.88 80.01 180)
-		(fields_autoplaced yes)
 		(effects
 			(font
@@
 		(shape bidirectional)
 		(at 182.88 82.55 180)
-		(fields_autoplaced yes)
-		(effects
-			(font
-				(size 1.27 1.27)
-			)
-			(justify right)
+		(effects
+			(font
+				(size 1.27 1.27)
+			)
+			(justify right)
+		)
+	)
+	(hierarchical_label "PA11"
+		(shape bidirectional)
+		(at 208.28 82.55 0)
+		(effects
+			(font
+				(size 1.27 1.27)
+			)
+			(justify left)
 		)
 	)
@@
 		(shape bidirectional)
 		(at 182.88 87.63 180)
-		(fields_autoplaced yes)
 		(effects
 			(font
@@
 		(shape bidirectional)
 		(at 208.28 54.61 0)
-		(fields_autoplaced yes)
 		(effects
 			(font
@@
 		(shape bidirectional)
 		(at 182.88 77.47 180)
-		(fields_autoplaced yes)
 		(effects
 			(font
@@
 		(shape bidirectional)
 		(at 208.28 80.01 0)
-		(fields_autoplaced yes)
 		(effects
 			(font
@@
 		(shape input)
 		(at 236.22 39.37 0)
-		(fields_autoplaced yes)
 		(effects
 			(font
@@
 		(shape input)
 		(at 55.88 30.48 180)
-		(fields_autoplaced yes)
 		(effects
 			(font
@@
 		(shape bidirectional)
 		(at 208.28 57.15 0)
-		(fields_autoplaced yes)
 		(effects
 			(font
@@
 		(shape bidirectional)
 		(at 208.28 69.85 0)
-		(fields_autoplaced yes)
-		(effects
-			(font
+		(effects
+			(font

Commit message: can transceiver and battery reverse polarity bypass
Parts:
- J10: footprint Connector_PinHeader_2.54mm:PinHeader_1x05_P2.54mm_Vertical -> Rocketry_Easyeda:CONN-SMD_5P-P1.25_532610571-2
- renumbered R26 to R27
Changed lines of the file:
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@@
 	(label "SWDIO"
 		(at 123.19 36.83 0)
+		(fields_autoplaced yes)
 		(effects
 			(font
@@
 	(label "GND"
 		(at 123.19 34.29 0)
+		(fields_autoplaced yes)
 		(effects
 			(font
@@
 	(label "GND"
 		(at 227.33 53.34 180)
+		(fields_autoplaced yes)
 		(effects
 			(font
@@
 	(label "SWDIO"
 		(at 208.28 87.63 0)
+		(fields_autoplaced yes)
 		(effects
 			(font
@@
 	(label "GND"
 		(at 195.58 104.14 180)
+		(fields_autoplaced yes)
 		(effects
 			(font
@@
 	(label "GND"
 		(at 157.48 54.61 180)
+		(fields_autoplaced yes)
 		(effects
 			(font
@@
 	(label "nRST"
 		(at 182.88 54.61 180)
+		(fields_autoplaced yes)
 		(effects
 			(font
@@
 	(label "SWDCLK"
 		(at 123.19 41.91 0)
+		(fields_autoplaced yes)
 		(effects
 			(font
@@
 	(label "GND"
 		(at 165.1 59.69 180)
+		(fields_autoplaced yes)
 		(effects
 			(font
@@
 	(label "nRST"
 		(at 123.19 31.75 0)
+		(fields_autoplaced yes)
 		(effects
 			(font
@@
 	(label "SWDCLK"
 		(at 208.28 90.17 0)
+		(fields_autoplaced yes)
 		(effects
 			(font
@@
 	(label "GND"
 		(at 55.88 30.48 0)
+		(fields_autoplaced yes)
 		(effects
 			(font
@@
 		(shape bidirectional)
 		(at 208.28 77.47 0)
+		(fields_autoplaced yes)
 		(effects
 			(font
@@
 		(shape bidirectional)
 		(at 182.88 72.39 180)
+		(fields_autoplaced yes)
 		(effects
 			(font
@@
 		(shape bidirectional)
 		(at 208.28 62.23 0)
+		(fields_autoplaced yes)
 		(effects
 			(font
@@
 		(shape bidirectional)
 		(at 182.88 74.93 180)
+		(fields_autoplaced yes)
 		(effects
 			(font
@@
 		(shape bidirectional)
 		(at 208.28 59.69 0)
+		(fields_autoplaced yes)
 		(effects
 			(font
@@
 		(shape bidirectional)
 		(at 208.28 64.77 0)
+		(fields_autoplaced yes)
 		(effects
 			(font
@@
 		(shape bidirectional)
 		(at 208.28 72.39 0)
+		(fields_autoplaced yes)
 		(effects
 			(font
@@
 		(shape input)
 		(at 142.24 35.56 180)
+		(fields_autoplaced yes)
 		(effects
 			(font
@@
 		(shape bidirectional)
 		(at 182.88 85.09 180)
+		(fields_autoplaced yes)
 		(effects
 			(font
@@
 		(shape bidirectional)
 		(at 208.28 67.31 0)
+		(fields_autoplaced yes)
 		(effects
 			(font
@@
 		(shape bidirectional)
 		(at 208.28 85.09 0)
+		(fields_autoplaced yes)
 		(effects
 			(font
@@
 		(shape bidirectional)
 		(at 182.88 80.01 180)
+		(fields_autoplaced yes)
 		(effects
 			(font
@@
 		(shape bidirectional)
 		(at 182.88 82.55 180)
+		(fields_autoplaced yes)
 		(effects
 			(font
@@
 		(shape bidirectional)
 		(at 208.28 82.55 0)
+		(fields_autoplaced yes)
 		(effects
 			(font
@@
 		(shape bidirectional)
 		(at 182.88 87.63 180)
+		(fields_autoplaced yes)
 		(effects
 			(font
@@
 		(shape bidirectional)
 		(at 208.28 54.61 0)
+		(fields_autoplaced yes)
 		(effects
 			(font
@@
 		(shape bidirectional)
 		(at 182.88 77.47 180)
+		(fields_autoplaced yes)
 		(effects
 			(font
@@
 		(shape bidirectional)
 		(at 208.28 80.01 0)
+		(fields_autoplaced yes)
 		(effects
 			(font
@@
 		(shape input)
 		(at 236.22 39.37 0)
+		(fields_autoplaced yes)
 		(effects
 			(font
@@
 		(shape input)
 		(at 55.88 30.48 180)
+		(fields_autoplaced yes)
 		(effects
 			(font
@@
 		(shape bidirectional)
 		(at 208.28 57.15 0)
+		(fields_autoplaced yes)
 		(effects
 			(font
@@
 		(shape bidirectional)
 		(at 208.28 69.85 0)
+		(fields_autoplaced yes)
 		(effects
 			(font
@@
 			)
 		)
-		(property "Footprint" "Connector_PinHeader_2.54mm:PinHeader_1x05_P2.54mm_Vertical"
+		(property "Footprint" "Rocketry_Easyeda:CONN-SMD_5P-P1.25_532610571-2"
 			(at 118.11 36.83 0)
 			(effects
@@
 		(dnp no)
 		(fields_autoplaced yes)
-		(property "Reference" "R26"
+		(property "Reference" "R27"
 			(at 171.45 53.34 0)
 			(effects
@@
 			(project "EPSv2"
 				(path "/61d36b12-c329-4dd2-b08b-b63678fc7b25/cef003e9-4e09-46ce-a170-d9263c8f93eb"
-					(reference "R26")
+					(reference "R27")
 					(unit 1)
 				)
