File: v2/blocks/TPS63070_5V.kicad_sch (KiCad schematic)
At the start: 15 parts, among them U24 1.5uF 2.9A, U25 TPS63070RNMR

Commit message: preliminary layout
Parts:
- renumbered U24 to L3, R39 to R33, R37 to R34, R38 to R35, R39 to R36, R40 to R37, U25 to U12
Changed lines of the file:
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@@
 		(dnp no)
 		(fields_autoplaced yes)
-		(property "Reference" "R40"
+		(property "Reference" "R37"
 			(at 168.91 90.17 90)
 			(effects
@@
 			(project ""
 				(path "/61d36b12-c329-4dd2-b08b-b63678fc7b25/6e2a5fe0-429e-4076-8476-90590336a78a"
-					(reference "R40")
+					(reference "R37")
 					(unit 1)
 				)
@@
 		(dnp no)
 		(fields_autoplaced yes)
-		(property "Reference" "R38"
+		(property "Reference" "R35"
 			(at 137.16 97.79 90)
 			(effects
@@
 			(project ""
 				(path "/61d36b12-c329-4dd2-b08b-b63678fc7b25/6e2a5fe0-429e-4076-8476-90590336a78a"
-					(reference "R38")
+					(reference "R35")
 					(unit 1)
 				)
@@
 					(unit 1)
 				)
-				(path "/61d36b12-c329-4dd2-b08b-b63678fc7b25/af831d8b-582d-46cc-acd1-685ce56b6776"
-					(reference "C35")
-					(unit 1)
-				)
 			)
 		)
@@
 					(unit 1)
 				)
-				(path "/61d36b12-c329-4dd2-b08b-b63678fc7b25/af831d8b-582d-46cc-acd1-685ce56b6776"
-					(reference "C34")
-					(unit 1)
-				)
 			)
 		)
@@
 					(unit 1)
 				)
-				(path "/61d36b12-c329-4dd2-b08b-b63678fc7b25/af831d8b-582d-46cc-acd1-685ce56b6776"
-					(reference "C32")
-					(unit 1)
-				)
 			)
 		)
@@
 					(unit 1)
 				)
-				(path "/61d36b12-c329-4dd2-b08b-b63678fc7b25/af831d8b-582d-46cc-acd1-685ce56b6776"
-					(reference "C30")
-					(unit 1)
-				)
 			)
 		)
@@
 					(unit 1)
 				)
-				(path "/61d36b12-c329-4dd2-b08b-b63678fc7b25/af831d8b-582d-46cc-acd1-685ce56b6776"
-					(reference "C33")
-					(unit 1)
-				)
 			)
 		)
@@
 		(dnp no)
 		(fields_autoplaced yes)
-		(property "Reference" "R39"
+		(property "Reference" "R36"
 			(at 154.94 95.25 90)
 			(effects
@@
 			(project ""
 				(path "/61d36b12-c329-4dd2-b08b-b63678fc7b25/6e2a5fe0-429e-4076-8476-90590336a78a"
-					(reference "R39")
+					(reference "R36")
 					(unit 1)
 				)
@@
 		(dnp no)
 		(fields_autoplaced yes)
-		(property "Reference" "R37"
+		(property "Reference" "R34"
 			(at 137.16 87.63 90)
 			(effects
@@
 			(project ""
 				(path "/61d36b12-c329-4dd2-b08b-b63678fc7b25/6e2a5fe0-429e-4076-8476-90590336a78a"
-					(reference "R37")
+					(reference "R34")
 					(unit 1)
 				)
@@
 		(on_board yes)
 		(dnp no)
-		(property "Reference" "R39"
+		(property "Reference" "R33"
 			(at 74.93 100.3299 90)
 			(effects
@@
 			(project "EPSv2"
 				(path "/61d36b12-c329-4dd2-b08b-b63678fc7b25/6e2a5fe0-429e-4076-8476-90590336a78a"
-					(reference "R36")
-					(unit 1)
-				)
-				(path "/61d36b12-c329-4dd2-b08b-b63678fc7b25/af831d8b-582d-46cc-acd1-685ce56b6776"
-					(reference "R39")
+					(reference "R33")
 					(unit 1)
 				)
@@
 		(dnp no)
 		(fields_autoplaced yes)
-		(property "Reference" "U25"
+		(property "Reference" "U12"
 			(at 104.14 90.17 0)
 			(effects
@@
 			(project "EPSv2"
 				(path "/61d36b12-c329-4dd2-b08b-b63678fc7b25/6e2a5fe0-429e-4076-8476-90590336a78a"
-					(reference "U13")
-					(unit 1)
-				)
-				(path "/61d36b12-c329-4dd2-b08b-b63678fc7b25/af831d8b-582d-46cc-acd1-685ce56b6776"
-					(reference "U25")
+					(reference "U12")
 					(unit 1)
 				)
@@
 					(unit 1)
 				)
-				(path "/61d36b12-c329-4dd2-b08b-b63678fc7b25/af831d8b-582d-46cc-acd1-685ce56b6776"
-					(reference "C31")
-					(unit 1)
-				)
 			)
 		)
@@
 		(dnp no)
 		(fields_autoplaced yes)
-		(property "Reference" "U24"
+		(property "Reference" "L3"
 			(at 104.14 76.2 0)
 			(effects
@@
 				(path "/61d36b12-c329-4dd2-b08b-b63678fc7b25/6e2a5fe0-429e-4076-8476-90590336a78a"
 					(reference "L3")
-					(unit 1)
-				)
-				(path "/61d36b12-c329-4dd2-b08b-b63678fc7b25/af831d8b-582d-46cc-acd1-685ce56b6776"
-					(reference "U24")
 					(unit 1)
 				)
@@
 					(reference "C36")
 					(unit 1)
-				)
-				(path "/61d36b12-c329-4dd2-b08b-b63678fc7b25/af831d8b-582d-46cc-acd1-685ce56b6776"
-					(reference "C36")
-					(unit 1)

Commit message: battery charging routing
Parts:
- renumbered C30 to C22, C31 to C23, C32 to C24, C33 to C25, C34 to C26, C35 to C27, C36 to C28
Changed lines of the file:
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@@
 		(dnp no)
 		(fields_autoplaced yes)
-		(property "Reference" "C35"
+		(property "Reference" "C27"
 			(at 212.09 87.6299 90)
 			(effects
@@
 			(project "EPSv2"
 				(path "/61d36b12-c329-4dd2-b08b-b63678fc7b25/6e2a5fe0-429e-4076-8476-90590336a78a"
-					(reference "C35")
+					(reference "C27")
 					(unit 1)
 				)
@@
 		(dnp no)
 		(fields_autoplaced yes)
-		(property "Reference" "C34"
+		(property "Reference" "C26"
 			(at 194.31 87.6299 90)
 			(effects
@@
 			(project "EPSv2"
 				(path "/61d36b12-c329-4dd2-b08b-b63678fc7b25/6e2a5fe0-429e-4076-8476-90590336a78a"
-					(reference "C34")
+					(reference "C26")
 					(unit 1)
 				)
@@
 		(on_board yes)
 		(dnp no)
-		(property "Reference" "C32"
+		(property "Reference" "C24"
 			(at 68.4746 87.6299 90)
 			(effects
@@
 			(project "EPSv2"
 				(path "/61d36b12-c329-4dd2-b08b-b63678fc7b25/6e2a5fe0-429e-4076-8476-90590336a78a"
-					(reference "C32")
+					(reference "C24")
 					(unit 1)
 				)
@@
 		(on_board yes)
 		(dnp no)
-		(property "Reference" "C30"
+		(property "Reference" "C22"
 			(at 32.8994 87.6299 90)
 			(effects
@@
 			(project "EPSv2"
 				(path "/61d36b12-c329-4dd2-b08b-b63678fc7b25/6e2a5fe0-429e-4076-8476-90590336a78a"
-					(reference "C30")
+					(reference "C22")
 					(unit 1)
 				)
@@
 		(on_board yes)
 		(dnp no)
-		(property "Reference" "C33"
+		(property "Reference" "C25"
 			(at 86.36 120.6499 90)
 			(effects
@@
 			(project "EPSv2"
 				(path "/61d36b12-c329-4dd2-b08b-b63678fc7b25/6e2a5fe0-429e-4076-8476-90590336a78a"
-					(reference "C33")
+					(reference "C25")
 					(unit 1)
 				)
@@
 		(on_board yes)
 		(dnp no)
-		(property "Reference" "C31"
+		(property "Reference" "C23"
 			(at 50.8 87.6299 90)
 			(effects
@@
 			(project "EPSv2"
 				(path "/61d36b12-c329-4dd2-b08b-b63678fc7b25/6e2a5fe0-429e-4076-8476-90590336a78a"
-					(reference "C31")
+					(reference "C23")
 					(unit 1)
 				)
@@
 		(dnp no)
 		(fields_autoplaced yes)
-		(property "Reference" "C36"
+		(property "Reference" "C28"
 			(at 229.87 87.6299 90)
 			(effects
@@
 			(project "EPSv2"
 				(path "/61d36b12-c329-4dd2-b08b-b63678fc7b25/6e2a5fe0-429e-4076-8476-90590336a78a"
-					(reference "C36")
-					(unit 1)
-				)
+					(reference "C28")
+					(unit 1)
+				)

Commit message: routing done
Parts:
- renumbered C22 to C24, C23 to C25, C24 to C26, C25 to C27, C26 to C28, C27 to C29, C28 to C30, R33 to R34, R34 to R35, R35 to R36, R36 to R37, R37 to R38, U12 to U10
Changed lines of the file:
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@@
 		(dnp no)
 		(fields_autoplaced yes)
-		(property "Reference" "R37"
+		(property "Reference" "R38"
 			(at 168.91 90.17 90)
 			(effects
@@
 			(project ""
 				(path "/61d36b12-c329-4dd2-b08b-b63678fc7b25/6e2a5fe0-429e-4076-8476-90590336a78a"
-					(reference "R37")
+					(reference "R38")
 					(unit 1)
 				)
@@
 		(dnp no)
 		(fields_autoplaced yes)
-		(property "Reference" "R35"
+		(property "Reference" "R36"
 			(at 137.16 97.79 90)
 			(effects
@@
 			(project ""
 				(path "/61d36b12-c329-4dd2-b08b-b63678fc7b25/6e2a5fe0-429e-4076-8476-90590336a78a"
-					(reference "R35")
+					(reference "R36")
 					(unit 1)
 				)
@@
 		(dnp no)
 		(fields_autoplaced yes)
-		(property "Reference" "C27"
+		(property "Reference" "C29"
 			(at 212.09 87.6299 90)
 			(effects
@@
 			(project "EPSv2"
 				(path "/61d36b12-c329-4dd2-b08b-b63678fc7b25/6e2a5fe0-429e-4076-8476-90590336a78a"
-					(reference "C27")
+					(reference "C29")
 					(unit 1)
 				)
@@
 		(dnp no)
 		(fields_autoplaced yes)
-		(property "Reference" "C26"
+		(property "Reference" "C28"
 			(at 194.31 87.6299 90)
 			(effects
@@
 			(project "EPSv2"
 				(path "/61d36b12-c329-4dd2-b08b-b63678fc7b25/6e2a5fe0-429e-4076-8476-90590336a78a"
-					(reference "C26")
+					(reference "C28")
 					(unit 1)
 				)
@@
 		(on_board yes)
 		(dnp no)
-		(property "Reference" "C24"
+		(property "Reference" "C26"
 			(at 68.4746 87.6299 90)
 			(effects
@@
 			(project "EPSv2"
 				(path "/61d36b12-c329-4dd2-b08b-b63678fc7b25/6e2a5fe0-429e-4076-8476-90590336a78a"
-					(reference "C24")
+					(reference "C26")
 					(unit 1)
 				)
@@
 		(on_board yes)
 		(dnp no)
-		(property "Reference" "C22"
+		(property "Reference" "C24"
 			(at 32.8994 87.6299 90)
 			(effects
@@
 			(project "EPSv2"
 				(path "/61d36b12-c329-4dd2-b08b-b63678fc7b25/6e2a5fe0-429e-4076-8476-90590336a78a"
-					(reference "C22")
+					(reference "C24")
 					(unit 1)
 				)
@@
 		(on_board yes)
 		(dnp no)
-		(property "Reference" "C25"
+		(property "Reference" "C27"
 			(at 86.36 120.6499 90)
 			(effects
@@
 			(project "EPSv2"
 				(path "/61d36b12-c329-4dd2-b08b-b63678fc7b25/6e2a5fe0-429e-4076-8476-90590336a78a"
-					(reference "C25")
+					(reference "C27")
 					(unit 1)
 				)
@@
 		(dnp no)
 		(fields_autoplaced yes)
-		(property "Reference" "R36"
+		(property "Reference" "R37"
 			(at 154.94 95.25 90)
 			(effects
@@
 			(project ""
 				(path "/61d36b12-c329-4dd2-b08b-b63678fc7b25/6e2a5fe0-429e-4076-8476-90590336a78a"
-					(reference "R36")
+					(reference "R37")
 					(unit 1)
 				)
@@
 		(dnp no)
 		(fields_autoplaced yes)
-		(property "Reference" "R34"
+		(property "Reference" "R35"
 			(at 137.16 87.63 90)
 			(effects
@@
 			(project ""
 				(path "/61d36b12-c329-4dd2-b08b-b63678fc7b25/6e2a5fe0-429e-4076-8476-90590336a78a"
-					(reference "R34")
+					(reference "R35")
 					(unit 1)
 				)
@@
 		(on_board yes)
 		(dnp no)
-		(property "Reference" "R33"
+		(property "Reference" "R34"
 			(at 74.93 100.3299 90)
 			(effects
@@
 			(project "EPSv2"
 				(path "/61d36b12-c329-4dd2-b08b-b63678fc7b25/6e2a5fe0-429e-4076-8476-90590336a78a"
-					(reference "R33")
+					(reference "R34")
 					(unit 1)
 				)
@@
 		(dnp no)
 		(fields_autoplaced yes)
-		(property "Reference" "U12"
+		(property "Reference" "U10"
 			(at 104.14 90.17 0)
 			(effects
@@
 			(project "EPSv2"
 				(path "/61d36b12-c329-4dd2-b08b-b63678fc7b25/6e2a5fe0-429e-4076-8476-90590336a78a"
-					(reference "U12")
+					(reference "U10")
 					(unit 1)
 				)
@@
 		(on_board yes)
 		(dnp no)
-		(property "Reference" "C23"
+		(property "Reference" "C25"
 			(at 50.8 87.6299 90)
 			(effects
@@
 			(project "EPSv2"
 				(path "/61d36b12-c329-4dd2-b08b-b63678fc7b25/6e2a5fe0-429e-4076-8476-90590336a78a"
-					(reference "C23")
+					(reference "C25")
 					(unit 1)
 				)
@@
 		(dnp no)
 		(fields_autoplaced yes)
-		(property "Reference" "C28"
+		(property "Reference" "C30"
 			(at 229.87 87.6299 90)
 			(effects
@@
 			(project "EPSv2"
 				(path "/61d36b12-c329-4dd2-b08b-b63678fc7b25/6e2a5fe0-429e-4076-8476-90590336a78a"
-					(reference "C28")
-					(unit 1)
-				)
+					(reference "C30")
+					(unit 1)
+				)

Commit message: can transceiver and battery reverse polarity bypass
Parts:
- renumbered R34 to R35, R35 to R36, R36 to R37, R37 to R38, R38 to R39
Changed lines of the file:
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@@
 		(shape input)
 		(at 90.17 127 270)
+		(fields_autoplaced yes)
 		(effects
 			(font
@@
 		(shape input)
 		(at 90.17 101.6 180)
+		(fields_autoplaced yes)
 		(effects
 			(font
@@
 		(shape input)
 		(at 33.02 83.82 180)
+		(fields_autoplaced yes)
 		(effects
 			(font
@@
 		(shape input)
 		(at 166.37 109.22 270)
+		(fields_autoplaced yes)
 		(effects
 			(font
@@
 		(shape input)
 		(at 118.11 114.3 0)
+		(fields_autoplaced yes)
 		(effects
 			(font
@@
 		(shape input)
 		(at 118.11 104.14 0)
+		(fields_autoplaced yes)
 		(effects
 			(font
@@
 		(shape input)
 		(at 134.62 104.14 270)
+		(fields_autoplaced yes)
 		(effects
 			(font
@@
 		(shape input)
 		(at 36.83 93.98 270)
+		(fields_autoplaced yes)
 		(effects
 			(font
@@
 		(shape input)
 		(at 118.11 116.84 0)
+		(fields_autoplaced yes)
 		(effects
 			(font
@@
 		(shape output)
 		(at 241.3 83.82 0)
+		(fields_autoplaced yes)
 		(effects
 			(font
@@
 		(shape input)
 		(at 226.06 93.98 270)
+		(fields_autoplaced yes)
 		(effects
 			(font
@@
 		(dnp no)
 		(fields_autoplaced yes)
-		(property "Reference" "R38"
+		(property "Reference" "R39"
 			(at 168.91 90.17 90)
 			(effects
@@
 			(project ""
 				(path "/61d36b12-c329-4dd2-b08b-b63678fc7b25/6e2a5fe0-429e-4076-8476-90590336a78a"
-					(reference "R38")
+					(reference "R39")
 					(unit 1)
 				)
@@
 		(dnp no)
 		(fields_autoplaced yes)
-		(property "Reference" "R36"
+		(property "Reference" "R37"
 			(at 137.16 97.79 90)
 			(effects
@@
 			(project ""
 				(path "/61d36b12-c329-4dd2-b08b-b63678fc7b25/6e2a5fe0-429e-4076-8476-90590336a78a"
-					(reference "R36")
+					(reference "R37")
 					(unit 1)
 				)
@@
 		(dnp no)
 		(fields_autoplaced yes)
-		(property "Reference" "R37"
+		(property "Reference" "R38"
 			(at 154.94 95.25 90)
 			(effects
@@
 			(project ""
 				(path "/61d36b12-c329-4dd2-b08b-b63678fc7b25/6e2a5fe0-429e-4076-8476-90590336a78a"
-					(reference "R37")
+					(reference "R38")
 					(unit 1)
 				)
@@
 		(dnp no)
 		(fields_autoplaced yes)
-		(property "Reference" "R35"
+		(property "Reference" "R36"
 			(at 137.16 87.63 90)
 			(effects
@@
 			(project ""
 				(path "/61d36b12-c329-4dd2-b08b-b63678fc7b25/6e2a5fe0-429e-4076-8476-90590336a78a"
-					(reference "R35")
+					(reference "R36")
 					(unit 1)
 				)
@@
 		(on_board yes)
 		(dnp no)
-		(property "Reference" "R34"
+		(property "Reference" "R35"
 			(at 74.93 100.3299 90)
 			(effects
@@
 			(project "EPSv2"
 				(path "/61d36b12-c329-4dd2-b08b-b63678fc7b25/6e2a5fe0-429e-4076-8476-90590336a78a"
-					(reference "R34")
-					(unit 1)
-				)
+					(reference "R35")
+					(unit 1)
+				)
