File: v2/blocks/TPS63070_3.3V.kicad_sch (KiCad schematic)
At the start: 15 parts, among them U13 1.5uF 2.9A, U14 TPS63070RNMR

Commit message: preliminary layout
Parts:
- renumbered U13 to L2, R31 to R28, R32 to R29, R33 to R30, R34 to R31, R35 to R32, U14 to U11
Changed lines of the file:
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@@
 		(dnp no)
 		(fields_autoplaced yes)
-		(property "Reference" "U13"
+		(property "Reference" "L2"
 			(at 104.14 76.2 0)
 			(effects
@@
 		(dnp no)
 		(fields_autoplaced yes)
-		(property "Reference" "U14"
+		(property "Reference" "U11"
 			(at 104.14 90.17 0)
 			(effects
@@
 			(project ""
 				(path "/61d36b12-c329-4dd2-b08b-b63678fc7b25/3a491354-fd14-404f-bfe4-727900531387"
-					(reference "U12")
+					(reference "U11")
 					(unit 1)
 				)
@@
 		(dnp no)
 		(fields_autoplaced yes)
-		(property "Reference" "R34"
+		(property "Reference" "R31"
 			(at 154.94 95.25 90)
 			(effects
@@
 			(project "EPSv2"
 				(path "/61d36b12-c329-4dd2-b08b-b63678fc7b25/3a491354-fd14-404f-bfe4-727900531387"
-					(reference "R34")
+					(reference "R31")
 					(unit 1)
 				)
@@
 		(on_board yes)
 		(dnp no)
-		(property "Reference" "R31"
+		(property "Reference" "R28"
 			(at 74.93 100.3299 90)
 			(effects
@@
 			(project ""
 				(path "/61d36b12-c329-4dd2-b08b-b63678fc7b25/3a491354-fd14-404f-bfe4-727900531387"
-					(reference "R31")
+					(reference "R28")
 					(unit 1)
 				)
@@
 		(dnp no)
 		(fields_autoplaced yes)
-		(property "Reference" "R35"
+		(property "Reference" "R32"
 			(at 168.91 90.17 90)
 			(effects
@@
 			(project ""
 				(path "/61d36b12-c329-4dd2-b08b-b63678fc7b25/3a491354-fd14-404f-bfe4-727900531387"
-					(reference "R35")
+					(reference "R32")
 					(unit 1)
 				)
@@
 		(dnp no)
 		(fields_autoplaced yes)
-		(property "Reference" "R33"
+		(property "Reference" "R30"
 			(at 137.16 97.79 90)
 			(effects
@@
 			(project ""
 				(path "/61d36b12-c329-4dd2-b08b-b63678fc7b25/3a491354-fd14-404f-bfe4-727900531387"
-					(reference "R33")
+					(reference "R30")
 					(unit 1)
 				)
@@
 		(dnp no)
 		(fields_autoplaced yes)
-		(property "Reference" "R32"
+		(property "Reference" "R29"
 			(at 137.16 87.63 90)
 			(effects
@@
 			(project ""
 				(path "/61d36b12-c329-4dd2-b08b-b63678fc7b25/3a491354-fd14-404f-bfe4-727900531387"
-					(reference "R32")
-					(unit 1)
-				)
+					(reference "R29")
+					(unit 1)
+				)

Commit message: battery charging routing
Parts:
- renumbered C23 to C15, C24 to C16, C25 to C17, C26 to C18, C27 to C19, C28 to C20, C29 to C21
Changed lines of the file:
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@@
 		(on_board yes)
 		(dnp no)
-		(property "Reference" "C26"
+		(property "Reference" "C18"
 			(at 86.36 120.6499 90)
 			(effects
@@
 			(project ""
 				(path "/61d36b12-c329-4dd2-b08b-b63678fc7b25/3a491354-fd14-404f-bfe4-727900531387"
-					(reference "C26")
+					(reference "C18")
 					(unit 1)
 				)
@@
 		(on_board yes)
 		(dnp no)
-		(property "Reference" "C25"
+		(property "Reference" "C17"
 			(at 68.4746 87.6299 90)
 			(effects
@@
 			(project ""
 				(path "/61d36b12-c329-4dd2-b08b-b63678fc7b25/3a491354-fd14-404f-bfe4-727900531387"
-					(reference "C25")
+					(reference "C17")
 					(unit 1)
 				)
@@
 		(dnp no)
 		(fields_autoplaced yes)
-		(property "Reference" "C29"
+		(property "Reference" "C21"
 			(at 229.87 87.6299 90)
 			(effects
@@
 			(project ""
 				(path "/61d36b12-c329-4dd2-b08b-b63678fc7b25/3a491354-fd14-404f-bfe4-727900531387"
-					(reference "C29")
+					(reference "C21")
 					(unit 1)
 				)
@@
 		(dnp no)
 		(fields_autoplaced yes)
-		(property "Reference" "C27"
+		(property "Reference" "C19"
 			(at 194.31 87.6299 90)
 			(effects
@@
 			(project ""
 				(path "/61d36b12-c329-4dd2-b08b-b63678fc7b25/3a491354-fd14-404f-bfe4-727900531387"
-					(reference "C27")
+					(reference "C19")
 					(unit 1)
 				)
@@
 		(dnp no)
 		(fields_autoplaced yes)
-		(property "Reference" "C28"
+		(property "Reference" "C20"
 			(at 212.09 87.6299 90)
 			(effects
@@
 			(project ""
 				(path "/61d36b12-c329-4dd2-b08b-b63678fc7b25/3a491354-fd14-404f-bfe4-727900531387"
-					(reference "C28")
+					(reference "C20")
 					(unit 1)
 				)
@@
 		(on_board yes)
 		(dnp no)
-		(property "Reference" "C24"
+		(property "Reference" "C16"
 			(at 50.8 87.6299 90)
 			(effects
@@
 			(project ""
 				(path "/61d36b12-c329-4dd2-b08b-b63678fc7b25/3a491354-fd14-404f-bfe4-727900531387"
-					(reference "C24")
+					(reference "C16")
 					(unit 1)
 				)
@@
 		(on_board yes)
 		(dnp no)
-		(property "Reference" "C23"
+		(property "Reference" "C15"
 			(at 32.8994 87.6299 90)
 			(effects
@@
 			(project ""
 				(path "/61d36b12-c329-4dd2-b08b-b63678fc7b25/3a491354-fd14-404f-bfe4-727900531387"
-					(reference "C23")
-					(unit 1)
-				)
+					(reference "C15")
+					(unit 1)
+				)

Commit message: routing done
Parts:
- renumbered C15 to C17, C16 to C18, C17 to C19, C18 to C20, C19 to C21, C20 to C22, C21 to C23, R28 to R29, R29 to R30, R30 to R31, R31 to R32, R32 to R33, U11 to U9
Changed lines of the file:
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@@
 		(dnp no)
 		(fields_autoplaced yes)
-		(property "Reference" "U11"
+		(property "Reference" "U9"
 			(at 104.14 90.17 0)
 			(effects
@@
 			(project ""
 				(path "/61d36b12-c329-4dd2-b08b-b63678fc7b25/3a491354-fd14-404f-bfe4-727900531387"
-					(reference "U11")
+					(reference "U9")
 					(unit 1)
 				)
@@
 		(on_board yes)
 		(dnp no)
-		(property "Reference" "C18"
+		(property "Reference" "C20"
 			(at 86.36 120.6499 90)
 			(effects
@@
 			(project ""
 				(path "/61d36b12-c329-4dd2-b08b-b63678fc7b25/3a491354-fd14-404f-bfe4-727900531387"
-					(reference "C18")
+					(reference "C20")
 					(unit 1)
 				)
@@
 		(on_board yes)
 		(dnp no)
-		(property "Reference" "C17"
+		(property "Reference" "C19"
 			(at 68.4746 87.6299 90)
 			(effects
@@
 			(project ""
 				(path "/61d36b12-c329-4dd2-b08b-b63678fc7b25/3a491354-fd14-404f-bfe4-727900531387"
-					(reference "C17")
+					(reference "C19")
 					(unit 1)
 				)
@@
 		(dnp no)
 		(fields_autoplaced yes)
-		(property "Reference" "C21"
+		(property "Reference" "C23"
 			(at 229.87 87.6299 90)
 			(effects
@@
 			(project ""
 				(path "/61d36b12-c329-4dd2-b08b-b63678fc7b25/3a491354-fd14-404f-bfe4-727900531387"
-					(reference "C21")
+					(reference "C23")
 					(unit 1)
 				)
@@
 		(dnp no)
 		(fields_autoplaced yes)
-		(property "Reference" "C19"
+		(property "Reference" "C21"
 			(at 194.31 87.6299 90)
 			(effects
@@
 			(project ""
 				(path "/61d36b12-c329-4dd2-b08b-b63678fc7b25/3a491354-fd14-404f-bfe4-727900531387"
-					(reference "C19")
+					(reference "C21")
 					(unit 1)
 				)
@@
 		(dnp no)
 		(fields_autoplaced yes)
-		(property "Reference" "R31"
+		(property "Reference" "R32"
 			(at 154.94 95.25 90)
 			(effects
@@
 			(project "EPSv2"
 				(path "/61d36b12-c329-4dd2-b08b-b63678fc7b25/3a491354-fd14-404f-bfe4-727900531387"
-					(reference "R31")
+					(reference "R32")
 					(unit 1)
 				)
@@
 		(dnp no)
 		(fields_autoplaced yes)
-		(property "Reference" "C20"
+		(property "Reference" "C22"
 			(at 212.09 87.6299 90)
 			(effects
@@
 			(project ""
 				(path "/61d36b12-c329-4dd2-b08b-b63678fc7b25/3a491354-fd14-404f-bfe4-727900531387"
-					(reference "C20")
+					(reference "C22")
 					(unit 1)
 				)
@@
 		(on_board yes)
 		(dnp no)
-		(property "Reference" "C16"
+		(property "Reference" "C18"
 			(at 50.8 87.6299 90)
 			(effects
@@
 			(project ""
 				(path "/61d36b12-c329-4dd2-b08b-b63678fc7b25/3a491354-fd14-404f-bfe4-727900531387"
-					(reference "C16")
+					(reference "C18")
 					(unit 1)
 				)
@@
 		(on_board yes)
 		(dnp no)
-		(property "Reference" "R28"
+		(property "Reference" "R29"
 			(at 74.93 100.3299 90)
 			(effects
@@
 			(project ""
 				(path "/61d36b12-c329-4dd2-b08b-b63678fc7b25/3a491354-fd14-404f-bfe4-727900531387"
-					(reference "R28")
+					(reference "R29")
 					(unit 1)
 				)
@@
 		(dnp no)
 		(fields_autoplaced yes)
-		(property "Reference" "R32"
+		(property "Reference" "R33"
 			(at 168.91 90.17 90)
 			(effects
@@
 			(project ""
 				(path "/61d36b12-c329-4dd2-b08b-b63678fc7b25/3a491354-fd14-404f-bfe4-727900531387"
-					(reference "R32")
+					(reference "R33")
 					(unit 1)
 				)
@@
 		(on_board yes)
 		(dnp no)
-		(property "Reference" "C15"
+		(property "Reference" "C17"
 			(at 32.8994 87.6299 90)
 			(effects
@@
 			(project ""
 				(path "/61d36b12-c329-4dd2-b08b-b63678fc7b25/3a491354-fd14-404f-bfe4-727900531387"
-					(reference "C15")
+					(reference "C17")
 					(unit 1)
 				)
@@
 		(dnp no)
 		(fields_autoplaced yes)
-		(property "Reference" "R30"
+		(property "Reference" "R31"
 			(at 137.16 97.79 90)
 			(effects
@@
 			(project ""
 				(path "/61d36b12-c329-4dd2-b08b-b63678fc7b25/3a491354-fd14-404f-bfe4-727900531387"
-					(reference "R30")
+					(reference "R31")
 					(unit 1)
 				)
@@
 		(dnp no)
 		(fields_autoplaced yes)
-		(property "Reference" "R29"
+		(property "Reference" "R30"
 			(at 137.16 87.63 90)
 			(effects
@@
 			(project ""
 				(path "/61d36b12-c329-4dd2-b08b-b63678fc7b25/3a491354-fd14-404f-bfe4-727900531387"
-					(reference "R29")
-					(unit 1)
-				)
+					(reference "R30")
+					(unit 1)
+				)

Commit message: can transceiver and battery reverse polarity bypass
Parts:
- renumbered R29 to R30, R30 to R31, R31 to R32, R32 to R33, R33 to R34
Changed lines of the file:
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@@
 		(shape output)
 		(at 241.3 83.82 0)
+		(fields_autoplaced yes)
 		(effects
 			(font
@@
 		(shape input)
 		(at 118.11 104.14 0)
+		(fields_autoplaced yes)
 		(effects
 			(font
@@
 		(shape input)
 		(at 36.83 93.98 270)
+		(fields_autoplaced yes)
 		(effects
 			(font
@@
 		(shape input)
 		(at 90.17 127 270)
+		(fields_autoplaced yes)
 		(effects
 			(font
@@
 		(shape input)
 		(at 166.37 109.22 270)
+		(fields_autoplaced yes)
 		(effects
 			(font
@@
 		(shape input)
 		(at 90.17 101.6 180)
+		(fields_autoplaced yes)
 		(effects
 			(font
@@
 		(shape input)
 		(at 226.06 93.98 270)
+		(fields_autoplaced yes)
 		(effects
 			(font
@@
 		(shape input)
 		(at 118.11 114.3 0)
+		(fields_autoplaced yes)
 		(effects
 			(font
@@
 		(shape input)
 		(at 33.02 83.82 180)
+		(fields_autoplaced yes)
 		(effects
 			(font
@@
 		(shape input)
 		(at 118.11 116.84 0)
+		(fields_autoplaced yes)
 		(effects
 			(font
@@
 		(shape input)
 		(at 134.62 104.14 270)
+		(fields_autoplaced yes)
 		(effects
 			(font
@@
 		(dnp no)
 		(fields_autoplaced yes)
-		(property "Reference" "R32"
+		(property "Reference" "R33"
 			(at 154.94 95.25 90)
 			(effects
@@
 			(project "EPSv2"
 				(path "/61d36b12-c329-4dd2-b08b-b63678fc7b25/3a491354-fd14-404f-bfe4-727900531387"
-					(reference "R32")
+					(reference "R33")
 					(unit 1)
 				)
@@
 		(on_board yes)
 		(dnp no)
-		(property "Reference" "R29"
+		(property "Reference" "R30"
 			(at 74.93 100.3299 90)
 			(effects
@@
 			(project ""
 				(path "/61d36b12-c329-4dd2-b08b-b63678fc7b25/3a491354-fd14-404f-bfe4-727900531387"
-					(reference "R29")
+					(reference "R30")
 					(unit 1)
 				)
@@
 		(dnp no)
 		(fields_autoplaced yes)
-		(property "Reference" "R33"
+		(property "Reference" "R34"
 			(at 168.91 90.17 90)
 			(effects
@@
 			(project ""
 				(path "/61d36b12-c329-4dd2-b08b-b63678fc7b25/3a491354-fd14-404f-bfe4-727900531387"
-					(reference "R33")
+					(reference "R34")
 					(unit 1)
 				)
@@
 		(dnp no)
 		(fields_autoplaced yes)
-		(property "Reference" "R31"
+		(property "Reference" "R32"
 			(at 137.16 97.79 90)
 			(effects
@@
 			(project ""
 				(path "/61d36b12-c329-4dd2-b08b-b63678fc7b25/3a491354-fd14-404f-bfe4-727900531387"
-					(reference "R31")
+					(reference "R32")
 					(unit 1)
 				)
@@
 		(dnp no)
 		(fields_autoplaced yes)
-		(property "Reference" "R30"
+		(property "Reference" "R31"
 			(at 137.16 87.63 90)
 			(effects
@@
 			(project ""
 				(path "/61d36b12-c329-4dd2-b08b-b63678fc7b25/3a491354-fd14-404f-bfe4-727900531387"
-					(reference "R30")
-					(unit 1)
-				)
+					(reference "R31")
+					(unit 1)
+				)
