File: v2/blocks/TPS63070_9V.kicad_sch (KiCad schematic)
At the start: 16 parts, among them U13 1.5uF 2.9A, U14 TPS63070RNMR

Commit message: preliminary layout
Parts:
- renumbered R45 to R42, R46 to R43
Changed lines of the file:
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@@
 				)
 				(path "/61d36b12-c329-4dd2-b08b-b63678fc7b25/af831d8b-582d-46cc-acd1-685ce56b6776"
-					(reference "L4")
+					(reference "L7")
 					(unit 1)
 				)
@@
 				)
 				(path "/61d36b12-c329-4dd2-b08b-b63678fc7b25/af831d8b-582d-46cc-acd1-685ce56b6776"
-					(reference "R41")
+					(reference "R38")
 					(unit 1)
 				)
@@
 		(dnp no)
 		(fields_autoplaced yes)
-		(property "Reference" "R45"
+		(property "Reference" "R42"
 			(at 154.94 95.25 90)
 			(effects
@@
 			(project "EPSv2"
 				(path "/61d36b12-c329-4dd2-b08b-b63678fc7b25/af831d8b-582d-46cc-acd1-685ce56b6776"
-					(reference "R45")
+					(reference "R42")
 					(unit 1)
 				)
@@
 				)
 				(path "/61d36b12-c329-4dd2-b08b-b63678fc7b25/af831d8b-582d-46cc-acd1-685ce56b6776"
-					(reference "R43")
+					(reference "R40")
 					(unit 1)
 				)
@@
 				)
 				(path "/61d36b12-c329-4dd2-b08b-b63678fc7b25/af831d8b-582d-46cc-acd1-685ce56b6776"
-					(reference "U20")
+					(reference "U16")
 					(unit 1)
 				)
@@
 				)
 				(path "/61d36b12-c329-4dd2-b08b-b63678fc7b25/af831d8b-582d-46cc-acd1-685ce56b6776"
-					(reference "R44")
+					(reference "R41")
 					(unit 1)
 				)
@@
 				)
 				(path "/61d36b12-c329-4dd2-b08b-b63678fc7b25/af831d8b-582d-46cc-acd1-685ce56b6776"
-					(reference "R42")
+					(reference "R39")
 					(unit 1)
 				)
@@
 		(dnp no)
 		(fields_autoplaced yes)
-		(property "Reference" "R46"
+		(property "Reference" "R43"
 			(at 168.91 90.17 90)
 			(effects
@@
 			(project ""
 				(path "/61d36b12-c329-4dd2-b08b-b63678fc7b25/af831d8b-582d-46cc-acd1-685ce56b6776"
-					(reference "R46")
-					(unit 1)
-				)
+					(reference "R43")
+					(unit 1)
+				)

Commit message: routing done
Parts:
- renumbered R42 to R50, R43 to R51
Changed lines of the file:
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@@
 				)
 				(path "/61d36b12-c329-4dd2-b08b-b63678fc7b25/af831d8b-582d-46cc-acd1-685ce56b6776"
-					(reference "L7")
+					(reference "L4")
 					(unit 1)
 				)
@@
 				)
 				(path "/61d36b12-c329-4dd2-b08b-b63678fc7b25/af831d8b-582d-46cc-acd1-685ce56b6776"
-					(reference "R38")
+					(reference "R46")
 					(unit 1)
 				)
@@
 				)
 				(path "/61d36b12-c329-4dd2-b08b-b63678fc7b25/af831d8b-582d-46cc-acd1-685ce56b6776"
-					(reference "C37")
+					(reference "C38")
 					(unit 1)
 				)
@@
 				)
 				(path "/61d36b12-c329-4dd2-b08b-b63678fc7b25/af831d8b-582d-46cc-acd1-685ce56b6776"
-					(reference "C32")
+					(reference "C33")
 					(unit 1)
 				)
@@
 		(dnp no)
 		(fields_autoplaced yes)
-		(property "Reference" "R42"
+		(property "Reference" "R50"
 			(at 154.94 95.25 90)
 			(effects
@@
 			(project "EPSv2"
 				(path "/61d36b12-c329-4dd2-b08b-b63678fc7b25/af831d8b-582d-46cc-acd1-685ce56b6776"
-					(reference "R42")
+					(reference "R50")
 					(unit 1)
 				)
@@
 				)
 				(path "/61d36b12-c329-4dd2-b08b-b63678fc7b25/af831d8b-582d-46cc-acd1-685ce56b6776"
-					(reference "R40")
+					(reference "R48")
 					(unit 1)
 				)
@@
 				)
 				(path "/61d36b12-c329-4dd2-b08b-b63678fc7b25/af831d8b-582d-46cc-acd1-685ce56b6776"
-					(reference "U16")
+					(reference "U12")
 					(unit 1)
 				)
@@
 				)
 				(path "/61d36b12-c329-4dd2-b08b-b63678fc7b25/af831d8b-582d-46cc-acd1-685ce56b6776"
-					(reference "R41")
+					(reference "R49")
 					(unit 1)
 				)
@@
 				)
 				(path "/61d36b12-c329-4dd2-b08b-b63678fc7b25/af831d8b-582d-46cc-acd1-685ce56b6776"
-					(reference "C38")
+					(reference "C39")
 					(unit 1)
 				)
@@
 				)
 				(path "/61d36b12-c329-4dd2-b08b-b63678fc7b25/af831d8b-582d-46cc-acd1-685ce56b6776"
-					(reference "C36")
+					(reference "C37")
 					(unit 1)
 				)
@@
 				)
 				(path "/61d36b12-c329-4dd2-b08b-b63678fc7b25/af831d8b-582d-46cc-acd1-685ce56b6776"
-					(reference "C33")
+					(reference "C34")
 					(unit 1)
 				)
@@
 				)
 				(path "/61d36b12-c329-4dd2-b08b-b63678fc7b25/af831d8b-582d-46cc-acd1-685ce56b6776"
-					(reference "C34")
+					(reference "C35")
 					(unit 1)
 				)
@@
 				)
 				(path "/61d36b12-c329-4dd2-b08b-b63678fc7b25/af831d8b-582d-46cc-acd1-685ce56b6776"
-					(reference "R39")
+					(reference "R47")
 					(unit 1)
 				)
@@
 		(dnp no)
 		(fields_autoplaced yes)
-		(property "Reference" "R43"
+		(property "Reference" "R51"
 			(at 168.91 90.17 90)
 			(effects
@@
 			(project ""
 				(path "/61d36b12-c329-4dd2-b08b-b63678fc7b25/af831d8b-582d-46cc-acd1-685ce56b6776"
-					(reference "R43")
+					(reference "R51")
 					(unit 1)
 				)
@@
 				)
 				(path "/61d36b12-c329-4dd2-b08b-b63678fc7b25/af831d8b-582d-46cc-acd1-685ce56b6776"
-					(reference "C35")
-					(unit 1)
-				)
+					(reference "C36")
+					(unit 1)
+				)

Commit message: CAN txrx
Parts:
- renumbered R50 to R57, R51 to R58
Changed lines of the file:
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@@
 		(shape input)
 		(at 118.11 114.3 0)
-		(fields_autoplaced yes)
 		(effects
 			(font
@@
 		(shape output)
 		(at 248.92 83.82 0)
-		(fields_autoplaced yes)
 		(effects
 			(font
@@
 		(shape input)
 		(at 118.11 116.84 0)
-		(fields_autoplaced yes)
 		(effects
 			(font
@@
 		(shape input)
 		(at 166.37 109.22 270)
-		(fields_autoplaced yes)
 		(effects
 			(font
@@
 		(shape input)
 		(at 90.17 127 270)
-		(fields_autoplaced yes)
 		(effects
 			(font
@@
 		(shape input)
 		(at 233.68 93.98 270)
-		(fields_autoplaced yes)
 		(effects
 			(font
@@
 		(shape input)
 		(at 118.11 104.14 0)
-		(fields_autoplaced yes)
 		(effects
 			(font
@@
 		(shape input)
 		(at 90.17 101.6 180)
-		(fields_autoplaced yes)
 		(effects
 			(font
@@
 		(shape input)
 		(at 134.62 104.14 270)
-		(fields_autoplaced yes)
 		(effects
 			(font
@@
 		(shape input)
 		(at 36.83 93.98 270)
-		(fields_autoplaced yes)
 		(effects
 			(font
@@
 		(shape input)
 		(at 33.02 83.82 180)
-		(fields_autoplaced yes)
 		(effects
 			(font
@@
 				)
 				(path "/61d36b12-c329-4dd2-b08b-b63678fc7b25/af831d8b-582d-46cc-acd1-685ce56b6776"
-					(reference "R46")
+					(reference "R53")
 					(unit 1)
 				)
@@
 				)
 				(path "/61d36b12-c329-4dd2-b08b-b63678fc7b25/af831d8b-582d-46cc-acd1-685ce56b6776"
-					(reference "C38")
+					(reference "C40")
 					(unit 1)
 				)
@@
 				)
 				(path "/61d36b12-c329-4dd2-b08b-b63678fc7b25/af831d8b-582d-46cc-acd1-685ce56b6776"
-					(reference "C33")
+					(reference "C35")
 					(unit 1)
 				)
@@
 		(dnp no)
 		(fields_autoplaced yes)
-		(property "Reference" "R50"
+		(property "Reference" "R57"
 			(at 154.94 95.25 90)
 			(effects
@@
 			(project "EPSv2"
 				(path "/61d36b12-c329-4dd2-b08b-b63678fc7b25/af831d8b-582d-46cc-acd1-685ce56b6776"
-					(reference "R50")
+					(reference "R57")
 					(unit 1)
 				)
@@
 				)
 				(path "/61d36b12-c329-4dd2-b08b-b63678fc7b25/af831d8b-582d-46cc-acd1-685ce56b6776"
-					(reference "R48")
+					(reference "R55")
 					(unit 1)
 				)
@@
 				)
 				(path "/61d36b12-c329-4dd2-b08b-b63678fc7b25/af831d8b-582d-46cc-acd1-685ce56b6776"
-					(reference "U12")
+					(reference "U13")
 					(unit 1)
 				)
@@
 				)
 				(path "/61d36b12-c329-4dd2-b08b-b63678fc7b25/af831d8b-582d-46cc-acd1-685ce56b6776"
-					(reference "R49")
+					(reference "R56")
 					(unit 1)
 				)
@@
 				)
 				(path "/61d36b12-c329-4dd2-b08b-b63678fc7b25/af831d8b-582d-46cc-acd1-685ce56b6776"
-					(reference "C39")
+					(reference "C41")
 					(unit 1)
 				)
@@
 				)
 				(path "/61d36b12-c329-4dd2-b08b-b63678fc7b25/af831d8b-582d-46cc-acd1-685ce56b6776"
-					(reference "C37")
+					(reference "C39")
 					(unit 1)
 				)
@@
 				)
 				(path "/61d36b12-c329-4dd2-b08b-b63678fc7b25/af831d8b-582d-46cc-acd1-685ce56b6776"
-					(reference "C34")
+					(reference "C36")
 					(unit 1)
 				)
@@
 				)
 				(path "/61d36b12-c329-4dd2-b08b-b63678fc7b25/af831d8b-582d-46cc-acd1-685ce56b6776"
-					(reference "C35")
+					(reference "C37")
 					(unit 1)
 				)
@@
 				)
 				(path "/61d36b12-c329-4dd2-b08b-b63678fc7b25/af831d8b-582d-46cc-acd1-685ce56b6776"
-					(reference "R47")
+					(reference "R54")
 					(unit 1)
 				)
@@
 		(dnp no)
 		(fields_autoplaced yes)
-		(property "Reference" "R51"
+		(property "Reference" "R58"
 			(at 168.91 90.17 90)
 			(effects
@@
 			(project ""
 				(path "/61d36b12-c329-4dd2-b08b-b63678fc7b25/af831d8b-582d-46cc-acd1-685ce56b6776"
-					(reference "R51")
+					(reference "R58")
 					(unit 1)
 				)
@@
 				)
 				(path "/61d36b12-c329-4dd2-b08b-b63678fc7b25/af831d8b-582d-46cc-acd1-685ce56b6776"
-					(reference "C36")
-					(unit 1)
-				)
+					(reference "C38")
+					(unit 1)
+				)

Commit message: can transceiver and battery reverse polarity bypass
Parts:
- renumbered R57 to R58, R58 to R59
Changed lines of the file:
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@@
 		(shape input)
 		(at 118.11 114.3 0)
+		(fields_autoplaced yes)
 		(effects
 			(font
@@
 		(shape output)
 		(at 248.92 83.82 0)
+		(fields_autoplaced yes)
 		(effects
 			(font
@@
 		(shape input)
 		(at 118.11 116.84 0)
+		(fields_autoplaced yes)
 		(effects
 			(font
@@
 		(shape input)
 		(at 166.37 109.22 270)
+		(fields_autoplaced yes)
 		(effects
 			(font
@@
 		(shape input)
 		(at 90.17 127 270)
+		(fields_autoplaced yes)
 		(effects
 			(font
@@
 		(shape input)
 		(at 233.68 93.98 270)
+		(fields_autoplaced yes)
 		(effects
 			(font
@@
 		(shape input)
 		(at 118.11 104.14 0)
+		(fields_autoplaced yes)
 		(effects
 			(font
@@
 		(shape input)
 		(at 90.17 101.6 180)
+		(fields_autoplaced yes)
 		(effects
 			(font
@@
 		(shape input)
 		(at 134.62 104.14 270)
+		(fields_autoplaced yes)
 		(effects
 			(font
@@
 		(shape input)
 		(at 36.83 93.98 270)
+		(fields_autoplaced yes)
 		(effects
 			(font
@@
 		(shape input)
 		(at 33.02 83.82 180)
+		(fields_autoplaced yes)
 		(effects
 			(font
@@
 				)
 				(path "/61d36b12-c329-4dd2-b08b-b63678fc7b25/af831d8b-582d-46cc-acd1-685ce56b6776"
-					(reference "R53")
+					(reference "R54")
 					(unit 1)
 				)
@@
 		(dnp no)
 		(fields_autoplaced yes)
-		(property "Reference" "R57"
+		(property "Reference" "R58"
 			(at 154.94 95.25 90)
 			(effects
@@
 			(project "EPSv2"
 				(path "/61d36b12-c329-4dd2-b08b-b63678fc7b25/af831d8b-582d-46cc-acd1-685ce56b6776"
-					(reference "R57")
+					(reference "R58")
 					(unit 1)
 				)
@@
 				)
 				(path "/61d36b12-c329-4dd2-b08b-b63678fc7b25/af831d8b-582d-46cc-acd1-685ce56b6776"
-					(reference "R55")
+					(reference "R56")
 					(unit 1)
 				)
@@
 				)
 				(path "/61d36b12-c329-4dd2-b08b-b63678fc7b25/af831d8b-582d-46cc-acd1-685ce56b6776"
-					(reference "R56")
+					(reference "R57")
 					(unit 1)
 				)
@@
 				)
 				(path "/61d36b12-c329-4dd2-b08b-b63678fc7b25/af831d8b-582d-46cc-acd1-685ce56b6776"
-					(reference "R54")
+					(reference "R55")
 					(unit 1)
 				)
@@
 		(dnp no)
 		(fields_autoplaced yes)
-		(property "Reference" "R58"
+		(property "Reference" "R59"
 			(at 168.91 90.17 90)
 			(effects
@@
 			(project ""
 				(path "/61d36b12-c329-4dd2-b08b-b63678fc7b25/af831d8b-582d-46cc-acd1-685ce56b6776"
-					(reference "R58")
-					(unit 1)
-				)
+					(reference "R59")
+					(unit 1)
+				)
